File: pcb/computer/computer.kicad_pcb (KiCad board)
At the start: 4 copper layers, 150 x 150 mm, 213 parts, among them J1 Conn_01x09_Female, J2 Conn_01x02_Female, J3 Conn_01x08_Female, J4 Conn_01x02_Male, J5 Conn_01x03_Male, J6 Conn_01x13_Female, J7 Conn_01x20_Female, J8 Conn_01x08_Female, SW1 SW_Push, SW2 SW_Push, SW3 SW_Push, SW4 SW_DIP_x08, SW5 SW_DIP_x08, SW7 SW_Push, U1 NE555D, U10 IS62C256AL-45ULI-TR, U11 74LS245, U12 74LS00, U13 NE555D, U14 74LS245, U15 74LS173, U16 74LS173, U17 74LS157, U18 74LS157, U19 L7805, U2 74LS00, U20 74LS245, U21 74LS04, U22 74LS173, U23 74LS173, U24 74LS173, U25 74LS30, U26 74LS04, U27 74LS283, U28 74LS283, U29 74LS245, U3 74LS245, U30 74LS173, U31 74LS173, U32 74LS86, U33 74LS86, U34 74LS04, U35 74LS245, U36 74LS173, U37 74LS173, U38 74LS161, U39 AT28C64B-15PU, U4 NE555D, U40 74LS173, U41 74LS173, U42 AT28C64B-15PU, U43 AT28C64B-15PU, U44 74LS173, U45 74LS173, U5 74LS161, U6 74LS161, U7 NE555D, U8 74LS157, U9 74LS157

Commit message: Update on the pcb
Parts:
- added D100: LED_Small, LED_SMD:LED_0603_1608Metric, F.Cu at (194.8, 84.5)
- added D38: LED_Small, LED_SMD:LED_0603_1608Metric, F.Cu at (65.0, 65.8)
- added D39: LED_Small, LED_SMD:LED_0603_1608Metric, F.Cu at (63.2, 65.8)
- added D40: LED_Small, LED_SMD:LED_0603_1608Metric, F.Cu at (61.4, 65.8)
- added D41: LED_Small, LED_SMD:LED_0603_1608Metric, F.Cu at (59.6, 65.8)
- added D42: LED_Small, LED_SMD:LED_0603_1608Metric, F.Cu at (57.8, 65.8)
- added D43: LED_Small, LED_SMD:LED_0603_1608Metric, F.Cu at (56.0, 65.8)
- added D44: LED_Small, LED_SMD:LED_0603_1608Metric, F.Cu at (52.4, 65.8)
- added D45: LED_Small, LED_SMD:LED_0603_1608Metric, F.Cu at (54.2, 65.8)
- added D46: LED_Small, LED_SMD:LED_0603_1608Metric, F.Cu at (84.9, 86.0)
- added D47: LED_Small, LED_SMD:LED_0603_1608Metric, F.Cu at (83.1, 86.0)
- added D48: LED_Small, LED_SMD:LED_0603_1608Metric, F.Cu at (81.3, 86.0)
- added D49: LED_Small, LED_SMD:LED_0603_1608Metric, F.Cu at (79.5, 86.0)
- added D50: LED_Small, LED_SMD:LED_0603_1608Metric, F.Cu at (77.7, 86.0)
- added D51: LED_Small, LED_SMD:LED_0603_1608Metric, F.Cu at (75.9, 86.0)
- added D52: LED_Small, LED_SMD:LED_0603_1608Metric, F.Cu at (72.3, 86.0)
- added D53: LED_Small, LED_SMD:LED_0603_1608Metric, F.Cu at (74.1, 86.0)
- added D54: LED_Small, LED_SMD:LED_0603_1608Metric, F.Cu at (131.9, 77.2)
- added D55: LED_Small, LED_SMD:LED_0603_1608Metric, F.Cu at (130.1, 77.2)
- added D56: LED_Small, LED_SMD:LED_0603_1608Metric, F.Cu at (128.2, 77.2)
- added D57: LED_Small, LED_SMD:LED_0603_1608Metric, F.Cu at (126.2, 77.2)
- added D58: LED_Small, LED_SMD:LED_0603_1608Metric, F.Cu at (124.3, 77.2)
- added D59: LED_Small, LED_SMD:LED_0603_1608Metric, F.Cu at (122.4, 77.2)
- added D60: LED_Small, LED_SMD:LED_0603_1608Metric, F.Cu at (118.5, 77.2)
- added D61: LED_Small, LED_SMD:LED_0603_1608Metric, F.Cu at (120.5, 77.2)
- added D62: LED_Small, LED_SMD:LED_0603_1608Metric, F.Cu at (131.9, 58.0)
- added D63: LED_Small, LED_SMD:LED_0603_1608Metric, F.Cu at (130.1, 58.0)
- added D64: LED_Small, LED_SMD:LED_0603_1608Metric, F.Cu at (128.2, 58.0)
- added D65: LED_Small, LED_SMD:LED_0603_1608Metric, F.Cu at (126.2, 58.0)
- added D66: LED_Small, LED_SMD:LED_0603_1608Metric, F.Cu at (124.3, 58.0)
- added D67: LED_Small, LED_SMD:LED_0603_1608Metric, F.Cu at (122.4, 58.0)
- added D68: LED_Small, LED_SMD:LED_0603_1608Metric, F.Cu at (118.5, 58.0)
- added D69: LED_Small, LED_SMD:LED_0603_1608Metric, F.Cu at (120.5, 58.0)
- added D70: LED_Small, LED_SMD:LED_0603_1608Metric, F.Cu at (130.1, 129.0)
- added D71: LED_Small, LED_SMD:LED_0603_1608Metric, F.Cu at (128.2, 129.0)
- added D72: LED_Small, LED_SMD:LED_0603_1608Metric, F.Cu at (126.2, 129.0)
- added D73: LED_Small, LED_SMD:LED_0603_1608Metric, F.Cu at (124.3, 129.0)
- added D74: LED_Small, LED_SMD:LED_0603_1608Metric, F.Cu at (122.5, 129.0)
- added D75: LED_Small, LED_SMD:LED_0603_1608Metric, F.Cu at (120.5, 129.0)
- added D76: LED_Small, LED_SMD:LED_0603_1608Metric, F.Cu at (116.8, 129.0)
- added D77: LED_Small, LED_SMD:LED_0603_1608Metric, F.Cu at (118.7, 129.0)
- added D78: LED_Small, LED_SMD:LED_0603_1608Metric, F.Cu at (132.8, 129.0)
- added D79: LED_Small, LED_SMD:LED_0603_1608Metric, F.Cu at (134.7, 129.0)
- added D80: LED_Small, LED_SMD:LED_0603_1608Metric, F.Cu at (136.6, 129.0)
- added D81: LED_Small, LED_SMD:LED_0603_1608Metric, F.Cu at (190.8, 71.5)
- added D82: LED_Small, LED_SMD:LED_0603_1608Metric, F.Cu at (190.8, 74.1)
- added D83: LED_Small, LED_SMD:LED_0603_1608Metric, F.Cu at (194.8, 71.5)
- added D84: LED_Small, LED_SMD:LED_0603_1608Metric, F.Cu at (190.8, 76.7)
- added D85: LED_Small, LED_SMD:LED_0603_1608Metric, F.Cu at (194.8, 74.1)
- added D86: LED_Small, LED_SMD:LED_0603_1608Metric, F.Cu at (198.9, 71.5)
- added D87: LED_Small, LED_SMD:LED_0603_1608Metric, F.Cu at (190.8, 79.3)
- added D88: LED_Small, LED_SMD:LED_0603_1608Metric, F.Cu at (194.8, 76.7)
- added D89: LED_Small, LED_SMD:LED_0603_1608Metric, F.Cu at (198.9, 74.1)
- added D90: LED_Small, LED_SMD:LED_0603_1608Metric, F.Cu at (190.8, 81.9)
- added D91: LED_Small, LED_SMD:LED_0603_1608Metric, F.Cu at (202.9, 71.5)
- added D92: LED_Small, LED_SMD:LED_0603_1608Metric, F.Cu at (194.8, 79.3)
- added D93: LED_Small, LED_SMD:LED_0603_1608Metric, F.Cu at (198.9, 76.7)
- added D94: LED_Small, LED_SMD:LED_0603_1608Metric, F.Cu at (190.8, 84.5)
- added D95: LED_Small, LED_SMD:LED_0603_1608Metric, F.Cu at (202.9, 74.1)
- added D96: LED_Small, LED_SMD:LED_0603_1608Metric, F.Cu at (194.8, 81.9)
- added D97: LED_Small, LED_SMD:LED_0603_1608Metric, F.Cu at (207.0, 71.5)
- added D98: LED_Small, LED_SMD:LED_0603_1608Metric, F.Cu at (198.9, 79.3)
- added D99: LED_Small, LED_SMD:LED_0603_1608Metric, F.Cu at (202.9, 76.7)
- added R100: R_Small, Resistor_SMD:R_0603_1608Metric, F.Cu at (195.5, 108.1)
- added R101: R_Small, Resistor_SMD:R_0603_1608Metric, F.Cu at (199.5, 105.6)
- added R102: R_Small, Resistor_SMD:R_0603_1608Metric, F.Cu at (199.5, 108.1)
- added R103: R_Small, Resistor_SMD:R_0603_1608Metric, F.Cu at (173.3, 131.9)
- added R104: R_Small, Resistor_SMD:R_0603_1608Metric, F.Cu at (177.3, 129.3)
- added R105: R_Small, Resistor_SMD:R_0603_1608Metric, F.Cu at (177.3, 131.9)
- added R106: R_Small, Resistor_SMD:R_0603_1608Metric, F.Cu at (207.0, 74.1)
- added R107: R_Small, Resistor_SMD:R_0603_1608Metric, F.Cu at (198.9, 81.9)
- added R108: R_Small, Resistor_SMD:R_0603_1608Metric, F.Cu at (211.0, 71.5)
- added R109: R_Small, Resistor_SMD:R_0603_1608Metric, F.Cu at (202.9, 79.3)
- added R110: R_Small, Resistor_SMD:R_0603_1608Metric, F.Cu at (207.0, 76.6)
- added R111: R_Small, Resistor_SMD:R_0603_1608Metric, F.Cu at (198.9, 84.4)
- added R112: R_Small, Resistor_SMD:R_0603_1608Metric, F.Cu at (211.0, 74.1)
- added R113: R_Small, Resistor_SMD:R_0603_1608Metric, F.Cu at (202.9, 81.8)
- added R114: R_Small, Resistor_SMD:R_0603_1608Metric, F.Cu at (215.0, 71.5)
- added R115: R_Small, Resistor_SMD:R_0603_1608Metric, F.Cu at (207.0, 79.1)
- added R116: R_Small, Resistor_SMD:R_0603_1608Metric, F.Cu at (211.0, 76.6)
- added R117: R_Small, Resistor_SMD:R_0603_1608Metric, F.Cu at (202.9, 84.3)
- added R118: R_Small, Resistor_SMD:R_0603_1608Metric, F.Cu at (215.0, 74.0)
- added R119: R_Small, Resistor_SMD:R_0603_1608Metric, F.Cu at (206.9, 81.6)
- added R120: R_Small, Resistor_SMD:R_0603_1608Metric, F.Cu at (211.0, 79.1)
- added R121: R_Small, Resistor_SMD:R_0603_1608Metric, F.Cu at (215.0, 76.5)
- added R122: R_Small, Resistor_SMD:R_0603_1608Metric, F.Cu at (206.9, 84.1)
- added R123: R_Small, Resistor_SMD:R_0603_1608Metric, F.Cu at (210.9, 81.6)
- added R124: R_Small, Resistor_SMD:R_0603_1608Metric, F.Cu at (215.0, 79.0)
- added R125: R_Small, Resistor_SMD:R_0603_1608Metric, F.Cu at (210.9, 84.1)
- added R63: R_Small, Resistor_SMD:R_0603_1608Metric, B.Cu at (65.0, 65.8)
- added R64: R_Small, Resistor_SMD:R_0603_1608Metric, B.Cu at (63.2, 65.8)
- added R65: R_Small, Resistor_SMD:R_0603_1608Metric, B.Cu at (61.4, 65.8)
- added R66: R_Small, Resistor_SMD:R_0603_1608Metric, B.Cu at (59.6, 65.8)
- added R67: R_Small, Resistor_SMD:R_0603_1608Metric, B.Cu at (57.8, 65.8)
- added R68: R_Small, Resistor_SMD:R_0603_1608Metric, B.Cu at (56.0, 65.8)
- added R69: R_Small, Resistor_SMD:R_0603_1608Metric, B.Cu at (52.4, 65.8)
- added R70: R_Small, Resistor_SMD:R_0603_1608Metric, B.Cu at (54.2, 65.8)
- added R71: R_Small, Resistor_SMD:R_0603_1608Metric, B.Cu at (84.9, 86.0)
- added R72: R_Small, Resistor_SMD:R_0603_1608Metric, B.Cu at (83.1, 86.0)
- added R73: R_Small, Resistor_SMD:R_0603_1608Metric, B.Cu at (81.3, 86.0)
- added R74: R_Small, Resistor_SMD:R_0603_1608Metric, B.Cu at (79.5, 86.0)
- added R75: R_Small, Resistor_SMD:R_0603_1608Metric, B.Cu at (77.7, 86.0)
- added R76: R_Small, Resistor_SMD:R_0603_1608Metric, B.Cu at (75.9, 86.0)
- added R77: R_Small, Resistor_SMD:R_0603_1608Metric, B.Cu at (72.3, 86.0)
- added R78: R_Small, Resistor_SMD:R_0603_1608Metric, B.Cu at (74.1, 86.0)
- added R79: R_Small, Resistor_SMD:R_0603_1608Metric, B.Cu at (131.9, 77.2)
- added R80: R_Small, Resistor_SMD:R_0603_1608Metric, B.Cu at (130.1, 77.2)
- added R81: R_Small, Resistor_SMD:R_0603_1608Metric, B.Cu at (128.2, 77.2)
- added R82: R_Small, Resistor_SMD:R_0603_1608Metric, B.Cu at (126.2, 77.2)
- added R83: R_Small, Resistor_SMD:R_0603_1608Metric, B.Cu at (124.3, 77.2)
- added R84: R_Small, Resistor_SMD:R_0603_1608Metric, B.Cu at (122.4, 77.2)
- added R85: R_Small, Resistor_SMD:R_0603_1608Metric, B.Cu at (118.5, 77.2)
- added R86: R_Small, Resistor_SMD:R_0603_1608Metric, B.Cu at (120.5, 77.2)
- added R87: R_Small, Resistor_SMD:R_0603_1608Metric, B.Cu at (131.9, 58.0)
- added R88: R_Small, Resistor_SMD:R_0603_1608Metric, B.Cu at (130.1, 58.0)
- added R89: R_Small, Resistor_SMD:R_0603_1608Metric, B.Cu at (128.2, 58.0)
- added R90: R_Small, Resistor_SMD:R_0603_1608Metric, B.Cu at (126.2, 58.0)
- added R91: R_Small, Resistor_SMD:R_0603_1608Metric, B.Cu at (124.3, 58.0)
- added R92: R_Small, Resistor_SMD:R_0603_1608Metric, B.Cu at (122.4, 58.0)
- added R93: R_Small, Resistor_SMD:R_0603_1608Metric, B.Cu at (118.5, 58.0)
- added R94: R_Small, Resistor_SMD:R_0603_1608Metric, B.Cu at (120.5, 58.0)
- added R95: R_Small, Resistor_SMD:R_0603_1608Metric, F.Cu at (195.5, 103.0)
- added R96: R_Small, Resistor_SMD:R_0603_1608Metric, F.Cu at (199.6, 100.5)
- added R97: R_Small, Resistor_SMD:R_0603_1608Metric, F.Cu at (191.5, 108.2)
- added R98: R_Small, Resistor_SMD:R_0603_1608Metric, F.Cu at (195.5, 105.6)
- added R99: R_Small, Resistor_SMD:R_0603_1608Metric, F.Cu at (199.5, 103.0)
- R10, R11, R12, R13, R16, R17, R18, R19, R20, R21, R22, R23, R25, R26, R27, R28, R29, R30, R31, R32, R6, R7, R8, R9: moved to B.Cu
- moved J5 601.0 mm to (84.0, 138.6)
- moved JP1 581.7 mm to (88.3, 134.0), turned to 270 degrees
- moved J7 579.4 mm to (99.0, 137.6), turned to 90 degrees
- moved C42 552.6 mm to (81.5, 125.6), turned to 180 degrees
- moved U39 550.9 mm to (89.0, 117.2), turned to 180 degrees
- moved C43 538.9 mm to (100.2, 125.4), turned to 180 degrees
- moved U42 533.7 mm to (107.9, 117.2), turned to 180 degrees
- moved J6 533.2 mm to (143.9, 134.4), turned to 180 degrees
- moved C44 524.9 mm to (119.2, 125.5), turned to 180 degrees
- moved U43 517.8 mm to (126.8, 117.2), turned to 180 degrees
- moved U38 457.5 mm to (107.1, 101.8), turned to 270 degrees
- moved C41 449.9 mm to (113.2, 104.0), turned to 270 degrees
- moved U30 395.8 mm to (83.6, 101.9), turned to 90 degrees
- moved U40 384.4 mm to (94.6, 86.8), turned to 270 degrees
- moved U41 382.0 mm to (107.0, 86.8), turned to 270 degrees
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Connections:
- J8 pad 1: OUTPUT_REGISTER_OUT_0 -> OUTPUT_REGISTER_OUT_6
- J8 pad 2: OUTPUT_REGISTER_OUT_1 -> OUTPUT_REGISTER_OUT_7
- J8 pad 3: OUTPUT_REGISTER_OUT_2 -> OUTPUT_REGISTER_OUT_4
- J8 pad 4: OUTPUT_REGISTER_OUT_3 -> OUTPUT_REGISTER_OUT_5
- J8 pad 5: OUTPUT_REGISTER_OUT_4 -> OUTPUT_REGISTER_OUT_2
- J8 pad 6: OUTPUT_REGISTER_OUT_5 -> OUTPUT_REGISTER_OUT_3
- J8 pad 7: OUTPUT_REGISTER_OUT_6 -> OUTPUT_REGISTER_OUT_0
- J8 pad 8: OUTPUT_REGISTER_OUT_7 -> OUTPUT_REGISTER_OUT_1
- R4 pad 1: Net-(R4-Pad1) -> CONTROL_ROM_IO_14
- SW3 pad 1: Net-(R4-Pad1) -> CONTROL_ROM_IO_14
- SW4 pad 1: RAM_TO_SWITCH_0 -> RAM_TO_SWITCH_7
- SW4 pad 2: RAM_TO_SWITCH_1 -> RAM_TO_SWITCH_6
- SW4 pad 3: RAM_TO_SWITCH_2 -> RAM_TO_SWITCH_5
- SW4 pad 4: RAM_TO_SWITCH_3 -> RAM_TO_SWITCH_4
- SW4 pad 5: RAM_TO_SWITCH_4 -> RAM_TO_SWITCH_3
- SW4 pad 6: RAM_TO_SWITCH_5 -> RAM_TO_SWITCH_2
- SW4 pad 7: RAM_TO_SWITCH_6 -> RAM_TO_SWITCH_1
- SW4 pad 8: RAM_TO_SWITCH_7 -> RAM_TO_SWITCH_0
- SW5 pad 1: RAM_ADDR_TO_SWITCH_0 -> RAM_ADDR_TO_SWITCH_7
- SW5 pad 2: RAM_ADDR_TO_SWITCH_1 -> RAM_ADDR_TO_SWITCH_6
- SW5 pad 3: RAM_ADDR_TO_SWITCH_2 -> RAM_ADDR_TO_SWITCH_5
- SW5 pad 4: RAM_ADDR_TO_SWITCH_3 -> RAM_ADDR_TO_SWITCH_4
- SW5 pad 5: RAM_ADDR_TO_SWITCH_4 -> RAM_ADDR_TO_SWITCH_3
- SW5 pad 6: RAM_ADDR_TO_SWITCH_5 -> RAM_ADDR_TO_SWITCH_2
- SW5 pad 7: RAM_ADDR_TO_SWITCH_6 -> RAM_ADDR_TO_SWITCH_1
- SW5 pad 8: RAM_ADDR_TO_SWITCH_7 -> RAM_ADDR_TO_SWITCH_0
- U21 pad 11: ALU_OUT_4 -> ALU_OUT_3
- U21 pad 13: ALU_OUT_5 -> ALU_OUT_1
- U21 pad 3: ALU_OUT_1 -> ALU_OUT_2
- U21 pad 5: ALU_OUT_2 -> ALU_OUT_4
- U21 pad 9: ALU_OUT_3 -> ALU_OUT_5
- U25 pad 1: Net-(U21-Pad2) -> Net-(U21-Pad10)
- U25 pad 11: Net-(U25-Pad11) -> Net-(U21-Pad2)
- U25 pad 12: Net-(U25-Pad12) -> Net-(U21-Pad12)
- U25 pad 3: Net-(U21-Pad6) -> Net-(U21-Pad8)
- U25 pad 4: Net-(U21-Pad8) -> Net-(U21-Pad6)
- U25 pad 5: Net-(U21-Pad10) -> Net-(U25-Pad5)
- U25 pad 6: Net-(U21-Pad12) -> Net-(U25-Pad6)
- U26 pad 2: Net-(U25-Pad11) -> Net-(U25-Pad5)
- U26 pad 4: Net-(U25-Pad12) -> Net-(U25-Pad6)
- U30 pad 11: BUS_7 -> BUS_4
- U30 pad 12: BUS_6 -> BUS_5
- U30 pad 13: BUS_5 -> BUS_6
- U30 pad 14: BUS_4 -> BUS_7
- U30 pad 3: CONTROL_ROM_ADDR_7 -> CONTROL_ROM_ADDR_10
- U30 pad 4: CONTROL_ROM_ADDR_8 -> CONTROL_ROM_ADDR_9
- U30 pad 5: CONTROL_ROM_ADDR_9 -> CONTROL_ROM_ADDR_8
- U30 pad 6: CONTROL_ROM_ADDR_10 -> CONTROL_ROM_ADDR_7
- U31 pad 11: BUS_3 -> BUS_0
- U31 pad 12: BUS_2 -> BUS_1
- U31 pad 13: BUS_1 -> BUS_2
- U31 pad 14: BUS_0 -> BUS_3
- U31 pad 3: CONTROL_ROM_ADDR_3 -> CONTROL_ROM_ADDR_6
- U31 pad 4: CONTROL_ROM_ADDR_4 -> CONTROL_ROM_ADDR_5
- U31 pad 5: CONTROL_ROM_ADDR_5 -> CONTROL_ROM_ADDR_4
- U31 pad 6: CONTROL_ROM_ADDR_6 -> CONTROL_ROM_ADDR_3
- U8 pad 10: RAM_TO_SWITCH_2 -> RAM_TO_SWITCH_1
- U8 pad 11: RAM_TO_BUS_2 -> RAM_TO_BUS_1
- U8 pad 12: RAM_IO_3 -> RAM_IO_0
- U8 pad 13: RAM_TO_SWITCH_3 -> RAM_TO_SWITCH_0
- U8 pad 14: RAM_TO_BUS_3 -> RAM_TO_BUS_0
- U8 pad 2: RAM_TO_BUS_0 -> RAM_TO_BUS_3
- U8 pad 3: RAM_TO_SWITCH_0 -> RAM_TO_SWITCH_3
- U8 pad 4: RAM_IO_0 -> RAM_IO_3
- U8 pad 5: RAM_TO_BUS_1 -> RAM_TO_BUS_2
- U8 pad 6: RAM_TO_SWITCH_1 -> RAM_TO_SWITCH_2
- U8 pad 7: RAM_IO_1 -> RAM_IO_2
- U8 pad 9: RAM_IO_2 -> RAM_IO_1
- U9 pad 10: RAM_TO_SWITCH_6 -> RAM_TO_SWITCH_5
- U9 pad 11: RAM_TO_BUS_6 -> RAM_TO_BUS_5
- U9 pad 12: RAM_IO_7 -> RAM_IO_4
- U9 pad 13: RAM_TO_SWITCH_7 -> RAM_TO_SWITCH_4
- U9 pad 14: RAM_TO_BUS_7 -> RAM_TO_BUS_4
- U9 pad 2: RAM_TO_BUS_4 -> RAM_TO_BUS_7
- U9 pad 3: RAM_TO_SWITCH_4 -> RAM_TO_SWITCH_7
- U9 pad 4: RAM_IO_4 -> RAM_IO_7
- U9 pad 5: RAM_TO_BUS_5 -> RAM_TO_BUS_6
- U9 pad 6: RAM_TO_SWITCH_5 -> RAM_TO_SWITCH_6
- U9 pad 7: RAM_IO_5 -> RAM_IO_6
- U9 pad 9: RAM_IO_6 -> RAM_IO_5
Routing:
- net BUS_0: track 102.3 -> 305.0 mm, vias 0 -> 6
- net BUS_1: track 99.8 -> 302.4 mm, vias 0 -> 6
- net BUS_2: track 96.8 -> 290.8 mm, vias 0 -> 6
- net BUS_3: track 93.7 -> 287.3 mm, vias 0 -> 6
- net BUS_4: track 74.6 -> 244.9 mm, vias 0 -> 6
- net BUS_5: track 72.2 -> 239.2 mm, vias 0 -> 6
- net BUS_6: track 69.2 -> 231.8 mm, vias 0 -> 6
- net BUS_7: track 65.9 -> 225.2 mm, vias 0 -> 6
- net RAM_TO_SWITCH_0: track 0.00 -> 81.5 mm, vias 0 -> 2
- net ALU_OUT_7: track 0.00 -> 79.1 mm, vias 0 -> 3
- net RAM_TO_SWITCH_1: track 0.00 -> 75.1 mm, vias 0 -> 2
- net RAM_TO_SWITCH_2: track 0.00 -> 74.5 mm, vias 0 -> 2
- net RAM_IO_1: track 0.00 -> 74.1 mm
- net RAM_IO_2: track 0.00 -> 69.8 mm
- net RAM_IO_0: track 0.00 -> 69.8 mm
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Other:
- board size 150 x 150 mm -> 114.5 x 102 mm

Commit message: Update pcb2
Parts:
- added C50: 10n, Capacitor_SMD:C_0603_1608Metric, F.Cu at (83.0, 110.8)
- added C51: 10n, Capacitor_SMD:C_0603_1608Metric, F.Cu at (103.2, 110.8)
- added C52: 10n, Capacitor_SMD:C_0603_1608Metric, F.Cu at (123.2, 110.8)
- added D101: LED_Small, LED_SMD:LED_0603_1608Metric, F.Cu at (118.4, 129.0)
- added D102: LED_Small, LED_SMD:LED_0603_1608Metric, F.Cu at (116.5, 129.0)
- added R126: R_Small, Resistor_SMD:R_0603_1608Metric, B.Cu at (118.4, 129.0)
- added R127: R_Small, Resistor_SMD:R_0603_1608Metric, B.Cu at (116.5, 129.0)
- added U46: 74LS04, Package_SO:SOIC-14_3.9x8.7mm_P1.27mm, F.Cu at (121.4, 116.3)
- added U47: 74LS04, Package_SO:SOIC-14_3.9x8.7mm_P1.27mm, F.Cu at (101.5, 116.3)
- added U48: 74LS04, Package_SO:SOIC-14_3.9x8.7mm_P1.27mm, F.Cu at (81.1, 116.2)
- R100, R101, R102, R103, R104, R105, R106, R107, R108, R109, R110, R111, R112, R113, R114, R115, R116, R117, R118, R119, R120, R121, R122, R123, R124, R125, R95, R96, R97, R98, R99: moved to B.Cu
- U12, U2: footprint Package_SO:SO-14_5.3x10.2mm_P1.27mm -> Package_SO:SOIC-14_3.9x8.7mm_P1.27mm
- moved R124 143.7 mm to (80.2, 129.0), turned to 270 degrees
- moved R125 139.9 mm to (78.4, 129.0), turned to 270 degrees
- moved R121 137.7 mm to (87.7, 129.0), turned to 270 degrees
- moved R123 137.2 mm to (82.2, 129.0), turned to 270 degrees
- moved D97 135.8 mm to (84.0, 129.0), turned to 90 degrees
- moved R118 135.2 mm to (91.5, 129.0), turned to 270 degrees
- moved R120 134.7 mm to (85.8, 129.0), turned to 270 degrees
- moved D99 133.4 mm to (80.2, 129.0), turned to 90 degrees
- moved R122 130.9 mm to (84.0, 129.0), turned to 270 degrees
- moved R114 129.6 mm to (98.8, 129.0), turned to 270 degrees
- moved D95 129.3 mm to (85.8, 129.0), turned to 90 degrees
- moved R116 127.1 mm to (95.2, 129.0), turned to 270 degrees
- moved D98 126.9 mm to (82.2, 129.0), turned to 90 degrees
- moved R119 126.6 mm to (89.5, 129.0), turned to 270 degrees
- moved D100 124.7 mm to (78.4, 129.0), turned to 90 degrees
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Connections:
- D94 pad 2: CONTROL_ROM_IO_13 -> ALU_OUT
- D97 pad 2: ALU_OUT_I -> CONTROL_ROM_IO_16
- J1 pad 9: CONTROL_ROM_IO_14 -> RAM_IN_I
- J6 pad 1: CONTROL_ROM_ADDR_0 -> CONTROL_ROM_ADDR_12
- J6 pad 10: CONTROL_ROM_ADDR_9 -> CONTROL_ROM_ADDR_3
- J6 pad 11: CONTROL_ROM_ADDR_10 -> CONTROL_ROM_ADDR_2
- J6 pad 12: CONTROL_ROM_ADDR_11 -> CONTROL_ROM_ADDR_1
- J6 pad 13: CONTROL_ROM_ADDR_12 -> CONTROL_ROM_ADDR_0
- J6 pad 2: CONTROL_ROM_ADDR_1 -> CONTROL_ROM_ADDR_11
- J6 pad 3: CONTROL_ROM_ADDR_2 -> CONTROL_ROM_ADDR_10
- J6 pad 4: CONTROL_ROM_ADDR_3 -> CONTROL_ROM_ADDR_9
- J6 pad 5: CONTROL_ROM_ADDR_4 -> CONTROL_ROM_ADDR_8
- J6 pad 6: CONTROL_ROM_ADDR_5 -> CONTROL_ROM_ADDR_7
- J6 pad 8: CONTROL_ROM_ADDR_7 -> CONTROL_ROM_ADDR_5
- J6 pad 9: CONTROL_ROM_ADDR_8 -> CONTROL_ROM_ADDR_4
- J7 pad 1: CONTROL_ROM_IO_0 -> CONTROL_ROM_IO_19
- J7 pad 10: CONTROL_ROM_IO_9 -> CONTROL_ROM_IO_10
- J7 pad 11: CONTROL_ROM_IO_10 -> CONTROL_ROM_IO_9
- J7 pad 12: CONTROL_ROM_IO_11 -> CONTROL_ROM_IO_8
- J7 pad 13: CONTROL_ROM_IO_12 -> CONTROL_ROM_IO_7
- J7 pad 14: CONTROL_ROM_IO_13 -> CONTROL_ROM_IO_6
- J7 pad 15: CONTROL_ROM_IO_14 -> CONTROL_ROM_IO_5
- J7 pad 16: CONTROL_ROM_IO_15 -> CONTROL_ROM_IO_4
- J7 pad 17: ALU_OUT_I -> CONTROL_ROM_IO_3
- J7 pad 18: CONTROL_ROM_IO_17 -> CONTROL_ROM_IO_2
- J7 pad 19: CONTROL_ROM_IO_18 -> CONTROL_ROM_IO_1
- J7 pad 2: CONTROL_ROM_IO_1 -> CONTROL_ROM_IO_18
- J7 pad 20: CONTROL_ROM_IO_19 -> CONTROL_ROM_IO_0
- J7 pad 3: CONTROL_ROM_IO_2 -> CONTROL_ROM_IO_17
- J7 pad 4: CONTROL_ROM_IO_3 -> CONTROL_ROM_IO_16
- J7 pad 5: CONTROL_ROM_IO_4 -> CONTROL_ROM_IO_15
- J7 pad 6: CONTROL_ROM_IO_5 -> CONTROL_ROM_IO_14
- J7 pad 7: CONTROL_ROM_IO_6 -> ALU_OUT
- J7 pad 8: CONTROL_ROM_IO_7 -> CONTROL_ROM_IO_12
- J7 pad 9: CONTROL_ROM_IO_8 -> CONTROL_ROM_IO_11
- R117 pad 1: Net-(R117-Pad1) -> GND
- R4 pad 1: CONTROL_ROM_IO_14 -> RAM_IN_I
- SW3 pad 1: CONTROL_ROM_IO_14 -> RAM_IN_I
- U10 pad 22: CONTROL_ROM_IO_13 -> RAM_OUT_I
- U10 pad 27: CONTROL_ROM_IO_14 -> RAM_IN_I
- U11 pad 19: CONTROL_ROM_IO_15 -> RAM_IO_I
- U12 pad 10: CONTROL_ROM_IO_0 -> CONTROL_ROM_IO_15
- U12 pad 9: CONTROL_ROM_IO_0 -> CONTROL_ROM_IO_15
- U14 pad 19: CONTROL_ROM_IO_5 -> REGISTER_A_OUT_I
- U15 pad 10: CONTROL_ROM_IO_4 -> REGISTER_A_IN_I
- U15 pad 9: CONTROL_ROM_IO_4 -> REGISTER_A_IN_I
- U16 pad 10: CONTROL_ROM_IO_4 -> REGISTER_A_IN_I
- U16 pad 9: CONTROL_ROM_IO_4 -> REGISTER_A_IN_I
- U20 pad 19: CONTROL_ROM_IO_7 -> REGISTER_B_OUT_I
- U22 pad 10: CONTROL_ROM_IO_6 -> REGISTER_B_IN_I
- U22 pad 9: CONTROL_ROM_IO_6 -> REGISTER_B_IN_I
- U23 pad 10: CONTROL_ROM_IO_6 -> REGISTER_B_IN_I
- U23 pad 9: CONTROL_ROM_IO_6 -> REGISTER_B_IN_I
- U24 pad 10: CONTROL_ROM_IO_18 -> FLAG_REGISTER_IN_I
- U24 pad 9: CONTROL_ROM_IO_18 -> FLAG_REGISTER_IN_I
- U27 pad 7: CONTROL_ROM_IO_17 -> CONTROL_ROM_IO_14
- U3 pad 19: CONTROL_ROM_IO_3 -> PC_OUT_I
- U30 pad 10: CONTROL_ROM_IO_8 -> INSTRUCTION_REGISTER_IN_I
- U30 pad 9: CONTROL_ROM_IO_8 -> INSTRUCTION_REGISTER_IN_I
- U31 pad 10: CONTROL_ROM_IO_8 -> INSTRUCTION_REGISTER_IN_I
- U31 pad 9: CONTROL_ROM_IO_8 -> INSTRUCTION_REGISTER_IN_I
- U32 pad 10: CONTROL_ROM_IO_17 -> CONTROL_ROM_IO_14
- U32 pad 13: CONTROL_ROM_IO_17 -> CONTROL_ROM_IO_14
- U32 pad 2: CONTROL_ROM_IO_17 -> CONTROL_ROM_IO_14
- U32 pad 5: CONTROL_ROM_IO_17 -> CONTROL_ROM_IO_14
- U33 pad 10: CONTROL_ROM_IO_17 -> CONTROL_ROM_IO_14
- U33 pad 13: CONTROL_ROM_IO_17 -> CONTROL_ROM_IO_14
- U33 pad 2: CONTROL_ROM_IO_17 -> CONTROL_ROM_IO_14
- U33 pad 5: CONTROL_ROM_IO_17 -> CONTROL_ROM_IO_14
- U35 pad 19: CONTROL_ROM_IO_10 -> PARAMETER_REGISTER_OUT_I
- U36 pad 10: CONTROL_ROM_IO_9 -> PARAMETER_REGISTER_IN_I
- U36 pad 9: CONTROL_ROM_IO_9 -> PARAMETER_REGISTER_IN_I
- U37 pad 10: CONTROL_ROM_IO_9 -> PARAMETER_REGISTER_IN_I
- U37 pad 9: CONTROL_ROM_IO_9 -> PARAMETER_REGISTER_IN_I
- U38 pad 1: CONTROL_ROM_IO_19 -> UCOUNTER_RESET_I
- U40 pad 10: CONTROL_ROM_IO_11 -> MEM_ADDR_REGISTER_IN_I
- U40 pad 9: CONTROL_ROM_IO_11 -> MEM_ADDR_REGISTER_IN_I
- U41 pad 10: CONTROL_ROM_IO_11 -> MEM_ADDR_REGISTER_IN_I
- U41 pad 9: CONTROL_ROM_IO_11 -> MEM_ADDR_REGISTER_IN_I
- U42 pad 17: CONTROL_ROM_IO_13 -> ALU_OUT
- U43 pad 11: ALU_OUT_I -> CONTROL_ROM_IO_16
- U44 pad 10: CONTROL_ROM_IO_12 -> OUTPUT_REGISTER_IN_I
- U44 pad 9: CONTROL_ROM_IO_12 -> OUTPUT_REGISTER_IN_I
- U45 pad 10: CONTROL_ROM_IO_12 -> OUTPUT_REGISTER_IN_I
- U45 pad 9: CONTROL_ROM_IO_12 -> OUTPUT_REGISTER_IN_I
- U5 pad 10: CONTROL_ROM_IO_2 -> CONTROL_ROM_IO_3
- U5 pad 7: CONTROL_ROM_IO_2 -> CONTROL_ROM_IO_3
- U5 pad 9: CONTROL_ROM_IO_1 -> PC_LOAD_I
- U6 pad 10: CONTROL_ROM_IO_2 -> CONTROL_ROM_IO_3
- U6 pad 7: CONTROL_ROM_IO_2 -> CONTROL_ROM_IO_3
- U6 pad 9: CONTROL_ROM_IO_1 -> PC_LOAD_I
Routing:
- net CONTROL_ROM_IO_17: track 0.00 -> 106.4 mm, vias 0 -> 2
- net CONTROL_ROM_IO_0: track 0.00 -> 106.1 mm, vias 0 -> 3
- net CONTROL_ROM_IO_1: track 0.00 -> 105.8 mm, vias 0 -> 3
- net CONTROL_ROM_ADDR_11: track 0.00 -> 104.1 mm, vias 0 -> 6
- net CONTROL_ROM_IO_18: track 0.00 -> 104.0 mm, vias 0 -> 2
- net REGISTER_A_IN_I: track 0.00 -> 101.4 mm, vias 0 -> 3
- net CONTROL_ROM_IO_16: track 0.00 -> 100.3 mm, vias 0 -> 2
- net CONTROL_ROM_IO_3: track 0.00 -> 100.3 mm, vias 0 -> 5
- net CONTROL_ROM_IO_19: track 0.00 -> 96.7 mm, vias 0 -> 2
- net CONTROL_ROM_IO_2: track 0.00 -> 89.6 mm, vias 0 -> 2
- net CONTROL_ROM_IO_5: track 0.00 -> 80.7 mm, vias 0 -> 2
- net CONTROL_ROM_IO_7: track 0.00 -> 79.9 mm, vias 0 -> 2
- net CONTROL_ROM_IO_6: track 0.00 -> 76.8 mm, vias 0 -> 2
- net CONTROL_ROM_IO_4: track 0.00 -> 72.5 mm, vias 0 -> 2
- net CONTROL_ROM_ADDR_12: track 38.8 -> 103.5 mm, vias 0 -> 6
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
Commit message: Finished pcb2
Parts:
- added R128: R_Small, Resistor_SMD:R_0603_1608Metric, F.Cu at (141.9, 122.3)
- added R129: R_Small, Resistor_SMD:R_0603_1608Metric, F.Cu at (138.9, 113.5)
- moved R34 4.66 mm to (46.1, 43.6)
- moved D9 3.51 mm to (46.1, 47.4)
- moved R43 1.71 mm to (42.6, 76.0), turned to 180 degrees
- moved D18 1.27 mm to (39.4, 76.0)
- moved C25 0.56 mm to (53.5, 43.8)
- moved C26 0.56 mm to (53.5, 47.2)
- moved J4 0.56 mm to (49.5, 46.8)
- moved U19 0.56 mm to (61.1, 45.5)
Connections:
- C42 pad 1: +5V -> ROM_5V
- C43 pad 1: +5V -> ROM_5V
- C44 pad 1: +5V -> ROM_5V
- J5 pad 1: +5V -> GND
- J5 pad 3: GND -> Net-(J5-Pad3)
- JP1 pad 2: +5V -> ROM_5V
- JP1 pad 3: +5V -> Net-(J5-Pad3)
- U39 pad 22: +5V -> ROM_5V
- U39 pad 28: +5V -> ROM_5V
- U42 pad 22: +5V -> ROM_5V
- U42 pad 28: +5V -> ROM_5V
- U43 pad 22: +5V -> ROM_5V
- U43 pad 28: +5V -> ROM_5V
Routing:
- net RESET: track 0.00 -> 304.9 mm, vias 0 -> 17
- net CLK: track 0.00 -> 286.1 mm, vias 0 -> 12
- net CLK_I: track 0.00 -> 150.4 mm, vias 0 -> 2
- net GND: track 33.5 -> 181.8 mm, vias 13 -> 157
- net CONTROL_ROM_IO_14: track 39.4 -> 179.9 mm, vias 2 -> 12
- net RESET_I: track 14.0 -> 135.6 mm, vias 0 -> 2
- net RAM_IN_I: track 0.00 -> 119.7 mm, vias 0 -> 3
- net RAM_IO_I: track 0.00 -> 115.8 mm, vias 0 -> 2
- net CONTROL_ROM_IO_15: track 42.1 -> 155.3 mm, vias 2 -> 3
- net ROM_5V: track 0.00 -> 112.0 mm, vias 0 -> 6
- net REGISTER_A_OUT_I: track 0.00 -> 89.3 mm, vias 0 -> 2
- net +5V: track 70.2 -> 146.3 mm, vias 13 -> 83
- net CLK_SELECT: track 2.64 -> 72.3 mm
- net RAM_PROGRAM: track 0.00 -> 68.1 mm, vias 0 -> 5
- net RAM_OUT_I: track 0.00 -> 67.8 mm, vias 0 -> 2
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