File: pcb/computer/computer.sch (KiCad schematic (older format))
At the start: 213 parts, among them J1 Conn_01x09_Female, J2 Conn_01x02_Female, J3 Conn_01x08_Female, J4 Conn_01x02_Male, J5 Conn_01x03_Male, J6 Conn_01x13_Female, J7 Conn_01x20_Female, J8 Conn_01x08_Female, SW1 SW_Push, SW2 SW_Push, SW3 SW_Push, SW4 SW_DIP_x08, SW5 SW_DIP_x08, SW7 SW_Push, U1 NE555D, U10 IS62C256AL-45ULI-TR, U11 74LS245, U12 74LS00, U13 NE555D, U14 74LS245, U15 74LS173, U16 74LS173, U17 74LS157, U18 74LS157, U19 L7805, U2 74LS00, U20 74LS245, U21 74LS04, U22 74LS173, U23 74LS173, U24 74LS173, U25 74LS30, U26 74LS04, U27 74LS283, U28 74LS283, U29 74LS245, U3 74LS245, U30 74LS173, U31 74LS173, U32 74LS86, U33 74LS86, U34 74LS04, U35 74LS245, U36 74LS173, U37 74LS173, U38 74LS161, U39 AT28C64B-15PU, U4 NE555D, U40 74LS173, U41 74LS173, U42 AT28C64B-15PU, U43 AT28C64B-15PU, U44 74LS173, U45 74LS173, U5 74LS161, U6 74LS161, U7 NE555D, U8 74LS157, U9 74LS157

Commit message: Update on the pcb
Parts:
- added D100, D38, D39, D40, D41, D42, D43, D44, D45, D46, D47, D48, D49, D50, D51, D52, D53, D54, D55, D56, D57, D58, D59, D60, D61, D62, D63, D64, D65, D66, D67, D68, D69, D70, D71, D72, D73, D74, D75, D76, D77, D78, D79, D80, D81, D82, D83, D84, D85, D86, D87, D88, D89, D90, D91, D92, D93, D94, D95, D96, D97, D98, D99: LED_Small, LED_SMD:LED_0603_1608Metric, symbol Device:LED_Small
- added R100, R101, R102, R103, R104, R105, R106, R107, R108, R109, R110, R111, R112, R113, R114, R115, R116, R117, R118, R119, R120, R121, R122, R123, R124, R125, R63, R64, R65, R66, R67, R68, R69, R70, R71, R72, R73, R74, R75, R76, R77, R78, R79, R80, R81, R82, R83, R84, R85, R86, R87, R88, R89, R90, R91, R92, R93, R94, R95, R96, R97, R98, R99: R_Small, Resistor_SMD:R_0603_1608Metric, symbol Device:R_Small
- U39, U42, U43: symbol AT28C64B-15PU:AT28C64B-15PU -> computer-rescue:AT28C64B-15PU-AT28C64B-15PU
Connections:
- net ALU_OUT_0: now also D46.2 (A)
- net ALU_OUT_1: now also U21.13, D47.2 (A); no longer U21.3
- net ALU_OUT_2: now also U21.3, D48.2 (A); no longer U21.5
- net ALU_OUT_3: now also U21.11, D49.2 (A); no longer U21.9
- net ALU_OUT_4: now also U21.5, D50.2 (A); no longer U21.11
- net ALU_OUT_5: now also U21.9, D51.2 (A); no longer U21.13
- net ALU_OUT_6: now also D53.2 (A)
- net ALU_OUT_7: now also D52.2 (A)
- net ALU_OUT_I: now also D97.2 (A)
- net BUS_0: now also U31.11 (D3); no longer U31.14 (D0)
- net BUS_1: now also U31.12 (D2); no longer U31.13 (D1)
- net BUS_2: now also U31.13 (D1); no longer U31.12 (D2)
- net BUS_3: now also U31.14 (D0); no longer U31.11 (D3)
- net BUS_4: now also U30.11 (D3); no longer U30.14 (D0)
- net BUS_5: now also U30.12 (D2); no longer U30.13 (D1)
- net BUS_6: now also U30.13 (D1); no longer U30.12 (D2)
- net BUS_7: now also U30.14 (D0); no longer U30.11 (D3)
- net CONTROL_ROM_ADDR_0: now also D78.2 (A)
- net CONTROL_ROM_ADDR_1: now also D79.2 (A)
- net CONTROL_ROM_ADDR_10: now also U30.3 (Q0), D76.2 (A); no longer U30.6 (Q3)
- net CONTROL_ROM_ADDR_2: now also D80.2 (A)
- net CONTROL_ROM_ADDR_3: now also U31.6 (Q3), D70.2 (A); no longer U31.3 (Q0)
- net CONTROL_ROM_ADDR_4: now also U31.5 (Q2), D71.2 (A); no longer U31.4 (Q1)
- net CONTROL_ROM_ADDR_5: now also U31.4 (Q1), D72.2 (A); no longer U31.5 (Q2)
- net CONTROL_ROM_ADDR_6: now also U31.3 (Q0), D73.2 (A); no longer U31.6 (Q3)
- net CONTROL_ROM_ADDR_7: now also U30.6 (Q3), D74.2 (A); no longer U30.3 (Q0)
- net CONTROL_ROM_ADDR_8: now also U30.5 (Q2), D75.2 (A); no longer U30.4 (Q1)
- net CONTROL_ROM_ADDR_9: now also U30.4 (Q1), D77.2 (A); no longer U30.5 (Q2)
- net CONTROL_ROM_IO_0: now also D81.2 (A)
- net CONTROL_ROM_IO_1: now also D82.2 (A)
- net CONTROL_ROM_IO_10: now also D91.2 (A)
- net CONTROL_ROM_IO_11: now also D92.2 (A)
- net CONTROL_ROM_IO_12: now also D93.2 (A)
- net CONTROL_ROM_IO_13: now also D94.2 (A)
- net CONTROL_ROM_IO_14: now also R4.1, SW3.1, D96.2 (A)
- net CONTROL_ROM_IO_15: now also D95.2 (A)
- net CONTROL_ROM_IO_17: now also D98.2 (A)
- net CONTROL_ROM_IO_18: now also D99.2 (A)
- net CONTROL_ROM_IO_19: now also D100.2 (A)
- net CONTROL_ROM_IO_2: now also D83.2 (A)
- net CONTROL_ROM_IO_3: now also D84.2 (A)
- net CONTROL_ROM_IO_4: now also D85.2 (A)
- net CONTROL_ROM_IO_5: now also D86.2 (A)
- net CONTROL_ROM_IO_6: now also D88.2 (A)
- net CONTROL_ROM_IO_7: now also D87.2 (A)
- net CONTROL_ROM_IO_8: now also D89.2 (A)
- net CONTROL_ROM_IO_9: now also D90.2 (A)
- net GND: now also R100.1, R101.1, R102.1, R103.1, R104.1, R105.1, R106.1, R107.1, R108.1, R109.1, R110.1, R111.1, R112.1, R113.1, R114.1, R115.1, R116.1, R118.1, R119.1, R120.1, R121.1, R122.1, R123.1, R124.1, R125.1, R63.1, R64.1, R65.1, R66.1, R67.1, R68.1, R69.1, R70.1, R71.1, R72.1, R73.1, R74.1, R75.1, R76.1, R77.1, R78.1, R79.1, R80.1, R81.1, R82.1, R83.1, R84.1, R85.1, R86.1, R87.1, R88.1, R89.1, R90.1, R91.1, R92.1, R93.1, R94.1, R95.1, R96.1, R97.1, R98.1, R99.1
- net OUTPUT_REGISTER_OUT_0: now also J8.7 (Pin_7); no longer J8.1 (Pin_1)
- net OUTPUT_REGISTER_OUT_1: now also J8.8 (Pin_8); no longer J8.2 (Pin_2)
- net OUTPUT_REGISTER_OUT_2: now also J8.5 (Pin_5); no longer J8.3 (Pin_3)
- net OUTPUT_REGISTER_OUT_3: now also J8.6 (Pin_6); no longer J8.4 (Pin_4)
- net OUTPUT_REGISTER_OUT_4: now also J8.3 (Pin_3); no longer J8.5 (Pin_5)
- net OUTPUT_REGISTER_OUT_5: now also J8.4 (Pin_4); no longer J8.6 (Pin_6)
- net OUTPUT_REGISTER_OUT_6: now also J8.1 (Pin_1); no longer J8.7 (Pin_7)
- net OUTPUT_REGISTER_OUT_7: now also J8.2 (Pin_2); no longer J8.8 (Pin_8)
- net RAM_ADDR_IN_0: now also D54.2 (A)
- net RAM_ADDR_IN_1: now also D55.2 (A)
- net RAM_ADDR_IN_2: now also D56.2 (A)
- net RAM_ADDR_IN_3: now also D57.2 (A)
- net RAM_ADDR_IN_4: now also D58.2 (A)
- net RAM_ADDR_IN_5: now also D59.2 (A)
- net RAM_ADDR_IN_6: now also D61.2 (A)
- net RAM_ADDR_IN_7: now also D60.2 (A)
- net RAM_ADDR_TO_SWITCH_0: now also SW5.8; no longer SW5.1
- net RAM_ADDR_TO_SWITCH_1: now also SW5.7; no longer SW5.2
- net RAM_ADDR_TO_SWITCH_2: now also SW5.6; no longer SW5.3
- net RAM_ADDR_TO_SWITCH_3: now also SW5.5; no longer SW5.4
- net RAM_ADDR_TO_SWITCH_4: now also SW5.4; no longer SW5.5
- net RAM_ADDR_TO_SWITCH_5: now also SW5.3; no longer SW5.6
- net RAM_ADDR_TO_SWITCH_6: now also SW5.2; no longer SW5.7
- net RAM_ADDR_TO_SWITCH_7: now also SW5.1; no longer SW5.8
- net RAM_IO_0: now also U8.12 (Zd), D62.2 (A); no longer U8.4 (Za)
- net RAM_IO_1: now also U8.9 (Zc), D63.2 (A); no longer U8.7 (Zb)
- net RAM_IO_2: now also U8.7 (Zb), D64.2 (A); no longer U8.9 (Zc)
- net RAM_IO_3: now also U8.4 (Za), D65.2 (A); no longer U8.12 (Zd)
- net RAM_IO_4: now also U9.12 (Zd), D66.2 (A); no longer U9.4 (Za)
- net RAM_IO_5: now also U9.9 (Zc), D67.2 (A); no longer U9.7 (Zb)
- net RAM_IO_6: now also U9.7 (Zb), D69.2 (A); no longer U9.9 (Zc)
- net RAM_IO_7: now also U9.4 (Za), D68.2 (A); no longer U9.12 (Zd)
- net RAM_TO_BUS_0: now also U8.14 (I0d); no longer U8.2 (I0a)
- net RAM_TO_BUS_1: now also U8.11 (I0c); no longer U8.5 (I0b)
- net RAM_TO_BUS_2: now also U8.5 (I0b); no longer U8.11 (I0c)
- net RAM_TO_BUS_3: now also U8.2 (I0a); no longer U8.14 (I0d)
- net RAM_TO_BUS_4: now also U9.14 (I0d); no longer U9.2 (I0a)
- net RAM_TO_BUS_5: now also U9.11 (I0c); no longer U9.5 (I0b)
- net RAM_TO_BUS_6: now also U9.5 (I0b); no longer U9.11 (I0c)
- net RAM_TO_BUS_7: now also U9.2 (I0a); no longer U9.14 (I0d)
- net RAM_TO_SWITCH_0: now also SW4.8, U8.13 (I1d); no longer SW4.1, U8.3 (I1a)
- net RAM_TO_SWITCH_1: now also SW4.7, U8.10 (I1c); no longer SW4.2, U8.6 (I1b)
- net RAM_TO_SWITCH_2: now also SW4.6, U8.6 (I1b); no longer SW4.3, U8.10 (I1c)
- net RAM_TO_SWITCH_3: now also SW4.5, U8.3 (I1a); no longer SW4.4, U8.13 (I1d)
- net RAM_TO_SWITCH_4: now also SW4.4, U9.13 (I1d); no longer SW4.5, U9.3 (I1a)
- net RAM_TO_SWITCH_5: now also SW4.3, U9.10 (I1c); no longer SW4.6, U9.6 (I1b)
- net RAM_TO_SWITCH_6: now also SW4.2, U9.6 (I1b); no longer SW4.7, U9.10 (I1c)
- net RAM_TO_SWITCH_7: now also SW4.1, U9.3 (I1a); no longer SW4.8, U9.13 (I1d)
- net REGISTER_A_OUT_0: now also D38.2 (A)
- net REGISTER_A_OUT_1: now also D39.2 (A)
- net REGISTER_A_OUT_2: now also D40.2 (A)
- net REGISTER_A_OUT_3: now also D41.2 (A)
- net REGISTER_A_OUT_4: now also D42.2 (A)
- net REGISTER_A_OUT_5: now also D43.2 (A)
- net REGISTER_A_OUT_6: now also D45.2 (A)
- net REGISTER_A_OUT_7: now also D44.2 (A)
- net at U25.1: now also U21.10; no longer U21.2
- net at U25.11: now also U21.2; no longer U26.2
- net at U25.12: now also U21.12; no longer U26.4
- net at U25.3: now also U21.8; no longer U21.6
- net at U25.4: now also U21.6; no longer U21.8
- net at U25.5: now also U26.2; no longer U21.10
- net at U25.6: now also U26.4; no longer U21.12
- new net: D38.1 (K), R63.2
- new net: D39.1 (K), R64.2
- new net: D40.1 (K), R65.2
- new net: D41.1 (K), R66.2
- new net: D42.1 (K), R67.2
- new net: D43.1 (K), R68.2
- new net: D45.1 (K), R70.2
- new net: D44.1 (K), R69.2
- new net: D46.1 (K), R71.2
- new net: D47.1 (K), R72.2
- new net: D48.1 (K), R73.2
- new net: D49.1 (K), R74.2
- new net: D50.1 (K), R75.2
- new net: D51.1 (K), R76.2
- new net: D53.1 (K), R78.2
- new net: D52.1 (K), R77.2
- new net: D54.1 (K), R79.2
- new net: D55.1 (K), R80.2
- new net: D56.1 (K), R81.2
- new net: D57.1 (K), R82.2
- new net: D58.1 (K), R83.2
- new net: D59.1 (K), R84.2
- new net: D61.1 (K), R86.2
- new net: D60.1 (K), R85.2
- new net: D62.1 (K), R87.2
- new net: D63.1 (K), R88.2
- new net: D64.1 (K), R89.2
- new net: D65.1 (K), R90.2
- new net: D66.1 (K), R91.2
- new net: D67.1 (K), R92.2
- new net: D69.1 (K), R94.2
- new net: D68.1 (K), R93.2
- new net: D70.1 (K), R95.2
- new net: D71.1 (K), R96.2
- new net: D72.1 (K), R97.2
- new net: D73.1 (K), R98.2
- new net: D74.1 (K), R99.2
- new net: D75.1 (K), R100.2
- new net: D77.1 (K), R102.2
- new net: D76.1 (K), R101.2
- new net: D78.1 (K), R103.2
- new net: D79.1 (K), R104.2
- new net: D80.1 (K), R105.2
- new net: D81.1 (K), R106.2
- new net: D82.1 (K), R107.2
- new net: D83.1 (K), R108.2
- new net: D84.1 (K), R109.2
- new net: D85.1 (K), R110.2
- new net: D86.1 (K), R111.2
- new net: D88.1 (K), R113.2
- new net: D87.1 (K), R112.2
- new net: D89.1 (K), R114.2
- new net: D90.1 (K), R115.2
- new net: D91.1 (K), R116.2
- new net: D92.1 (K), R117.2
- new net: D93.1 (K), R118.2
- new net: D94.1 (K), R119.2
- new net: D96.1 (K), R121.2
- new net: D95.1 (K), R120.2
- new net: D97.1 (K), R122.2
- new net: D98.1 (K), R123.2
- new net: D99.1 (K), R124.2
- new net: D100.1 (K), R125.2
Other:
- moved on the sheet: C27, C28, C29, C37, C41, C42, C43, C44, C49, J5, J6, J7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

Commit message: Update pcb2
Parts:
- added C50, C51, C52: 10n, Capacitor_SMD:C_0603_1608Metric, symbol Device:C_Small
- added D101, D102: LED_Small, LED_SMD:LED_0603_1608Metric, symbol Device:LED_Small
- added R126, R127: R_Small, Resistor_SMD:R_0603_1608Metric, symbol Device:R_Small
- added U46, U47, U48: 74LS04, Package_SO:SOIC-14_3.9x8.7mm_P1.27mm, symbol 74xx:74LS04
Connections:
- net +5V: now also C50.1, C51.1, C52.1, U46.14 (VCC), U47.14 (VCC), U48.14 (VCC)
- net ALU_OUT_I: now also U47.6; no longer D97.2 (A), J7.17 (Pin_17), U43.11 (I/O0)
- net CONTROL_ROM_ADDR_0: now also J6.13 (Pin_13); no longer J6.1 (Pin_1)
- net CONTROL_ROM_ADDR_1: now also J6.12 (Pin_12); no longer J6.2 (Pin_2)
- net CONTROL_ROM_ADDR_10: now also J6.3 (Pin_3); no longer J6.11 (Pin_11)
- net CONTROL_ROM_ADDR_11: now also J6.2 (Pin_2), D101.2 (A); no longer J6.12 (Pin_12)
- net CONTROL_ROM_ADDR_12: now also J6.1 (Pin_1), D102.2 (A); no longer J6.13 (Pin_13)
- net CONTROL_ROM_ADDR_2: now also J6.11 (Pin_11); no longer J6.3 (Pin_3)
- net CONTROL_ROM_ADDR_3: now also J6.10 (Pin_10); no longer J6.4 (Pin_4)
- net CONTROL_ROM_ADDR_4: now also J6.9 (Pin_9); no longer J6.5 (Pin_5)
- net CONTROL_ROM_ADDR_5: now also J6.8 (Pin_8); no longer J6.6 (Pin_6)
- net CONTROL_ROM_ADDR_7: now also J6.6 (Pin_6); no longer J6.8 (Pin_8)
- net CONTROL_ROM_ADDR_8: now also J6.5 (Pin_5); no longer J6.9 (Pin_9)
- net CONTROL_ROM_ADDR_9: now also J6.4 (Pin_4); no longer J6.10 (Pin_10)
- net CONTROL_ROM_IO_0: now also J7.20 (Pin_20), U48.9; no longer J7.1 (Pin_1), U12.10, U12.9
- net CONTROL_ROM_IO_1: now also J7.19 (Pin_19), U48.11; no longer J7.2 (Pin_2), U5.9 (~PE), U6.9 (~PE)
- net CONTROL_ROM_IO_10: now also J7.10 (Pin_10), U46.1; no longer J7.11 (Pin_11), U35.19 (CE)
- net CONTROL_ROM_IO_11: now also J7.9 (Pin_9), U47.13; no longer J7.12 (Pin_12), U40.10 (E2), U40.9 (E1), U41.10 (E2), U41.9 (E1)
- net CONTROL_ROM_IO_12: now also J7.8 (Pin_8), U47.3; no longer J7.13 (Pin_13), U44.10 (E2), U44.9 (E1), U45.10 (E2), U45.9 (E1)
- net CONTROL_ROM_IO_14: now also J7.6 (Pin_6), U27.7 (C0), U32.10, U32.13, U32.2, U32.5, U33.10, U33.13, U33.2, U33.5; no longer J1.9 (Pin_9), J7.15 (Pin_15), R4.1, SW3.1, U10.27 (~WE~)
- net CONTROL_ROM_IO_15: now also J7.5 (Pin_5), U12.10, U12.9; no longer J7.16 (Pin_16), U11.19 (CE)
- net CONTROL_ROM_IO_17: now also J7.3 (Pin_3), U46.11; no longer J7.18 (Pin_18), U27.7 (C0), U32.10, U32.13, U32.2, U32.5, U33.10, U33.13, U33.2, U33.5
- net CONTROL_ROM_IO_18: now also J7.2 (Pin_2), U46.13; no longer J7.19 (Pin_19), U24.10 (E2), U24.9 (E1)
- net CONTROL_ROM_IO_19: now also J7.1 (Pin_1), U46.3; no longer J7.20 (Pin_20), U38.1 (~MR)
- net CONTROL_ROM_IO_2: now also J7.18 (Pin_18), U47.1; no longer J7.3 (Pin_3), U5.10 (CET), U5.7 (CEP), U6.10 (CET), U6.7 (CEP)
- net CONTROL_ROM_IO_3: now also J7.17 (Pin_17), U5.10 (CET), U5.7 (CEP), U6.10 (CET), U6.7 (CEP); no longer J7.4 (Pin_4), U3.19 (CE)
- net CONTROL_ROM_IO_4: now also J7.16 (Pin_16), U48.13; no longer J7.5 (Pin_5), U15.10 (E2), U15.9 (E1), U16.10 (E2), U16.9 (E1)
- net CONTROL_ROM_IO_5: now also J7.15 (Pin_15), U48.1; no longer J7.6 (Pin_6), U14.19 (CE)
- net CONTROL_ROM_IO_6: now also J7.14 (Pin_14), U48.3; no longer J7.7 (Pin_7), U22.10 (E2), U22.9 (E1), U23.10 (E2), U23.9 (E1)
- net CONTROL_ROM_IO_7: now also J7.13 (Pin_13), U48.5; no longer J7.8 (Pin_8), U20.19 (CE)
- net CONTROL_ROM_IO_8: now also J7.12 (Pin_12), U47.9; no longer J7.9 (Pin_9), U30.10 (E2), U30.9 (E1), U31.10 (E2), U31.9 (E1)
- net CONTROL_ROM_IO_9: now also J7.11 (Pin_11), U47.11; no longer J7.10 (Pin_10), U36.10 (E2), U36.9 (E1), U37.10 (E2), U37.9 (E1)
- net GND: now also R117.1, C50.2, C51.2, C52.2, R126.1, R127.1, U46.7 (GND), U47.7 (GND), U48.7 (GND)
- net CONTROL_ROM_IO_13 renamed ALU_OUT
- net ALU_OUT: now also J7.7 (Pin_7), U47.5; no longer J7.14 (Pin_14), U10.22 (~OE~)
- new net: D101.1 (K), R126.2
- new net: D102.1 (K), R127.2
- new net CONTROL_ROM_IO_16: D97.2 (A), J7.4 (Pin_4), U43.11 (I/O0), U46.9
- new net FLAG_REGISTER_IN_I: U24.10 (E2), U24.9 (E1), U47.2
- new net INSTRUCTION_REGISTER_IN_I: U30.10 (E2), U30.9 (E1), U31.10 (E2), U31.9 (E1), U47.8
- new net MEM_ADDR_REGISTER_IN_I: U40.10 (E2), U40.9 (E1), U41.10 (E2), U41.9 (E1), U47.10
- new net OUTPUT_REGISTER_IN_I: U44.10 (E2), U44.9 (E1), U45.10 (E2), U45.9 (E1), U46.8
- new net PARAMETER_REGISTER_IN_I: U36.10 (E2), U36.9 (E1), U37.10 (E2), U37.9 (E1), U48.4
- new net PARAMETER_REGISTER_OUT_I: U35.19 (CE), U48.6
- new net PC_LOAD_I: U48.12, U5.9 (~PE), U6.9 (~PE)
- new net PC_OUT_I: U3.19 (CE), U48.2
- new net RAM_IN_I: J1.9 (Pin_9), R4.1, SW3.1, U10.27 (~WE~), U46.12
- new net RAM_IO_I: U11.19 (CE), U46.2
- new net RAM_OUT_I: U10.22 (~OE~), U46.10
- new net REGISTER_A_IN_I: U15.10 (E2), U15.9 (E1), U16.10 (E2), U16.9 (E1), U47.4
- new net REGISTER_A_OUT_I: U14.19 (CE), U47.12
- new net REGISTER_B_IN_I: U22.10 (E2), U22.9 (E1), U23.10 (E2), U23.9 (E1), U48.10
- new net REGISTER_B_OUT_I: U20.19 (CE), U48.8
- new net UCOUNTER_RESET_I: U38.1 (~MR), U46.4

Commit message: Finished pcb2
Parts:
- added R128, R129: R_Small, Resistor_SMD:R_0603_1608Metric, symbol Device:R_Small
Connections:
- net +5V: now also R128.2; no longer C42.1, C43.1, C44.1, J5.1 (Pin_1), JP1.2, JP1.3, U39.22 (~OE~), U39.28 (VCC), U42.22 (~OE~), U42.28 (VCC), U43.22 (~OE~), U43.28 (VCC)
- net CONTROL_ROM_IN_I: now also R128.1
- net GND: now also J5.1 (Pin_1), R129.1; no longer J5.3 (Pin_3)
- new net: J5.3 (Pin_3), JP1.3
- new net ROM_5V: C42.1, C43.1, C44.1, JP1.2, R129.2, U39.22 (~OE~), U39.28 (VCC), U42.22 (~OE~), U42.28 (VCC), U43.22 (~OE~), U43.28 (VCC)
Other:
- moved on the sheet: C50, C51, C52, J5, JP1
