File: pcb/homebrew-computer/control_logic.sch (KiCad schematic (older format))
At the start: 0 parts

Commit message: Add part of the control logic
Parts:
- added C? (x7): 100n, symbol Device:C_Small
- added U? (x5): XC9536XL-10VQG44C, symbol XC9500XL:XC9536XL-10VQG44C
- added U? (x2): 74LVC16374ADGG,112, symbol 74LVC16374ADGG:74LVC16374ADGG,112
Connections:
- new net: C?.1, C?.1, C?.1, C?.1, U?.18 (VCC), U?.31 (VCC), U?.42 (VCC), U?.7 (VCC)
- new net +3V3: C?.1, C?.1, C?.1, U?.15 (VCCINT_3.3V), U?.26 (VCCIO_2.5V/3.3V), U?.35 (VCCINT_3.3V)
- new net DBUS1: U?.2 (1Q0), U?.47 (1D0)
- new net DBUS10: U?.14 (2Q1), U?.35 (2D1)
- new net DBUS11: U?.16 (2Q2), U?.33 (2D2)
- new net DBUS12: U?.17 (2Q3), U?.32 (2D3)
- new net DBUS13: U?.19 (2Q4), U?.30 (2D4)
- new net DBUS14: U?.20 (2Q5), U?.29 (2D5)
- new net DBUS15: U?.22 (2Q6), U?.27 (2D6)
- new net DBUS16: U?.23 (2Q7), U?.26 (2D7)
- new net DBUS2: U?.3 (1Q1), U?.46 (1D1)
- new net DBUS3: U?.44 (1D2), U?.5 (1Q2)
- new net DBUS4: U?.43 (1D3), U?.6 (1Q3)
- new net DBUS5: U?.41 (1D4), U?.8 (1Q4)
- new net DBUS6: U?.40 (1D5), U?.9 (1Q5)
- new net DBUS7: U?.11 (1Q6), U?.38 (1D6)
- new net DBUS8: U?.12 (1Q7), U?.37 (1D7)
- new net DBUS9: U?.13 (2Q0), U?.36 (2D0)
- new net GND: C?.2, C?.2, C?.2, C?.2, C?.2, C?.2, C?.2, U?.10 (GND), U?.15 (GND), U?.17 (GND), U?.21 (GND), U?.25 (GND), U?.28 (GND), U?.34 (GND), U?.39 (GND), U?.4 (GND), U?.4 (GND), U?.45 (GND)
- new net INSTR_IN: U?.25 (2CP), U?.48 (1CP)
- new net INSTR_OUT: U?.1 (1OE), U?.24 (2OE)
- new net TCK: U?.11 (TCK)
- new net TDI: U?.9 (TDI)
- new net TDO: U?.24 (TDO)
- new net TMS: U?.10 (TMS)
Other:
- note added: "Inputs/Outputs"
- note added: "Instruction register"
- note added: "JTAG"
- note added: "Power"
- note added: "Register"
