File: pcb/homebrew-computer/control_logic.sch (KiCad schematic (older format))
At the start: 13 parts, among them U14 XC95144XL-10TQ100C, U15 74LVC16374ADGG,112

Commit message: Keep working on the layout
Connections:
- net ALU_OUT_I: now also U14.90 (IO); no longer U14.14 (IO)
- net IR1: now also U14.91 (IO); no longer U14.90 (IO)
- net IR10: now also U14.4 (IO,GTS2); no longer U14.3 (IO,GTS1)
- net IR11: now also U14.6 (IO); no longer U14.4 (IO,GTS2)
- net IR12: now also U14.7 (IO); no longer U14.6 (IO)
- net IR13: now also U14.8 (IO); no longer U14.7 (IO)
- net IR14: now also U14.9 (IO); no longer U14.8 (IO)
- net IR15: now also U14.10 (IO); no longer U14.9 (IO)
- net IR16: now also U14.11 (IO); no longer U14.10 (IO)
- net IR2: now also U14.92 (IO); no longer U14.91 (IO)
- net IR3: now also U14.93 (IO); no longer U14.92 (IO)
- net IR4: now also U14.94 (IO); no longer U14.93 (IO)
- net IR5: now also U14.95 (IO); no longer U14.94 (IO)
- net IR6: now also U14.96 (IO); no longer U14.95 (IO)
- net IR7: now also U14.1 (IO,GTS3); no longer U14.96 (IO)
- net IR8: now also U14.2 (IO,GTS4); no longer U14.1 (IO,GTS3)
- net IR9: now also U14.3 (IO,GTS1); no longer U14.2 (IO,GTS4)
- net REG3_IN_L: no longer U14.11 (IO)
Changed lines of the file:
@@
 Text HLabel 8350 3350 2    50   Output ~ 0
 OP4
-Text HLabel 4350 2950 0    50   Output ~ 0
+Text HLabel 5800 4000 2    50   Output ~ 0
 ALU_OUT_I
 Text HLabel 8350 2950 2    50   Input ~ 0
@@
 Text HLabel 6900 3250 0    50   Output ~ 0
 REG3_IN_H
-Text HLabel 4350 2650 0    50   Output ~ 0
+Text HLabel 4050 2850 0    50   Output ~ 0
 REG3_IN_L
 Text HLabel 4350 4600 0    50   Output ~ 0
@@
 Text Label 2450 3900 0    50   ~ 0
 IR16
-Text Label 5800 4000 0    50   ~ 0
+Text Label 5800 4100 0    50   ~ 0
 IR1
-Text Label 5800 4100 0    50   ~ 0
+Text Label 5800 4200 0    50   ~ 0
 IR2
-Text Label 5800 4200 0    50   ~ 0
+Text Label 5800 4300 0    50   ~ 0
 IR3
-Text Label 5800 4300 0    50   ~ 0
+Text Label 5800 4400 0    50   ~ 0
 IR4
-Text Label 5800 4400 0    50   ~ 0
+Text Label 5800 4500 0    50   ~ 0
 IR5
-Text Label 5800 4500 0    50   ~ 0
+Text Label 5800 4600 0    50   ~ 0
 IR6
-Text Label 5800 4600 0    50   ~ 0
+Text Label 5800 2850 0    50   ~ 0
 IR7
-Text Label 5800 2850 0    50   ~ 0
+Text Label 5800 2950 0    50   ~ 0
 IR8
-Text Label 5800 2950 0    50   ~ 0
+Text Label 5800 3050 0    50   ~ 0
 IR9
-Text Label 5800 3050 0    50   ~ 0
+Text Label 5800 3150 0    50   ~ 0
 IR10
-Text Label 5800 3150 0    50   ~ 0
+Text Label 5800 3250 0    50   ~ 0
 IR11
-Text Label 5800 3250 0    50   ~ 0
+Text Label 5800 3350 0    50   ~ 0
 IR12
-Text Label 5800 3350 0    50   ~ 0
+Text Label 5800 3450 0    50   ~ 0
 IR13
-Text Label 5800 3450 0    50   ~ 0
+Text Label 5800 3550 0    50   ~ 0
 IR14
-Text Label 5800 3550 0    50   ~ 0
+Text Label 5800 3650 0    50   ~ 0
 IR15
-Text Label 5800 3650 0    50   ~ 0
+Text Label 4350 2650 2    50   ~ 0
 IR16
 Text Label 5800 4700 0    50   ~ 0

Commit message: Finished working on the layout
Connections:
- net INT: now also U14.66 (IO); no longer U14.50 (IO)
- net IO_ADDR_IN: now also U14.60 (IO); no longer U14.59 (IO)
- net IO_IN: now also U14.63 (IO); no longer U14.55 (IO)
- net IO_INB: now also U14.65 (IO); no longer U14.58 (IO)
- net IO_OUT: now also U14.61 (IO); no longer U14.54 (IO)
- net IO_OUTB: now also U14.64 (IO); no longer U14.56 (IO)
- net PERIPH_MEM_SPACE: now also U14.68 (IO); no longer U14.60 (IO)
- net REG1_IN_L: now also U14.17 (IO)
- net REG1_OUT_H_I: now also U14.18 (IO)
- net REG1_OUT_L_I: now also U14.16 (IO)
- net REG2_IN_H: now also U14.35 (IO)
- net REG2_IN_L: now also U14.43 (IO)
- net REG2_OUT_L_I: now also U14.42 (IO)
- net REG3_IN_H: now also U14.71 (IO); no longer U14.41 (IO)
- net REG3_IN_L: now also U14.54 (IO)
- net REG3_OUT_H_I: now also U14.70 (IO)
- net REG3_OUT_L_I: now also U14.53 (IO)
- net RST_INT: now also U14.67 (IO); no longer U14.53 (IO)
- no-connect marks 8 -> 21
Changed lines of the file:
@@
 Text HLabel 8350 3150 2    50   Input ~ 0
 FLAG_OVERFLOW
-Text HLabel 4100 3500 0    50   Input ~ 0
+Text HLabel 4350 3150 0    50   Input ~ 0
 REG1_OUT_L_I
-Text HLabel 4100 3200 0    50   Input ~ 0
+Text HLabel 4350 3350 0    50   Input ~ 0
 REG1_OUT_H_I
 Text HLabel 4350 4300 0    50   Output ~ 0
 REG1_IN_H
-Text HLabel 4100 3300 0    50   Output ~ 0
+Text HLabel 4350 3250 0    50   Output ~ 0
 REG1_IN_L
-Text HLabel 4100 3400 0    50   Output ~ 0
+Text HLabel 6900 3350 0    50   Output ~ 0
 REG2_OUT_L_I
 Text HLabel 4350 4200 0    50   Output ~ 0
 REG2_OUT_H_I
-Text HLabel 4100 3700 0    50   Output ~ 0
+Text HLabel 6900 2750 0    50   Output ~ 0
 REG2_IN_H
-Text HLabel 4100 3800 0    50   Output ~ 0
+Text HLabel 6900 3450 0    50   Output ~ 0
 REG2_IN_L
-Text HLabel 4100 3900 0    50   Output ~ 0
+Text HLabel 6900 4000 0    50   Output ~ 0
 REG3_OUT_L_I
-Text HLabel 4100 4000 0    50   Output ~ 0
+Text HLabel 8350 4400 2    50   Output ~ 0
 REG3_OUT_H_I
-Text HLabel 6900 3250 0    50   Output ~ 0
+Text HLabel 8350 4500 2    50   Output ~ 0
 REG3_IN_H
-Text HLabel 4050 2850 0    50   Output ~ 0
-REG3_IN_L
 Text HLabel 4350 4600 0    50   Output ~ 0
 SP_OUT_I
@@
 $Comp
 L XC9500XL:XC95144XL-10TQ100C U14
-U 6 1 5FA858A3
-P 4650 3600
-F 0 "U14" H 4650 2350 50  0000 R CNN
-F 1 "XC95144XL-10TQ100C" H 5200 2250 50  0000 R CNN
-F 2 "Package_QFP:TQFP-100_14x14mm_P0.5mm" H 4650 3600 50  0001 C CNN
-F 3 "" H 4650 3600 50  0001 C CNN
-	6    4650 3600
-	-1   0    0    -1
-$EndComp
-$Comp
-L XC9500XL:XC95144XL-10TQ100C U14
 U 8 1 5FA90592
 P 7250 2550
@@
 Text Notes 1250 4900 0    50   Italic 0
 The instruction register is always\noutputing its content to the control logic
-Text HLabel 6900 3800 0    50   Input ~ 0
+Text HLabel 8350 4100 2    50   Input ~ 0
 INT
-Text HLabel 6900 3900 0    50   Output ~ 0
-INT_OUT_I
-Text HLabel 6900 4000 0    50   Output ~ 0
+Text HLabel 8350 4200 2    50   Output ~ 0
 RST_INT
-Text HLabel 6900 4100 0    50   Output ~ 0
+Text HLabel 6900 4700 0    50   Output ~ 0
 IO_OUT
-Text HLabel 6900 4200 0    50   Output ~ 0
+Text HLabel 8350 3800 2    50   Output ~ 0
 IO_IN
-Text HLabel 6900 4300 0    50   Output ~ 0
+Text HLabel 8350 3900 2    50   Output ~ 0
 IO_OUTB
-Text HLabel 6900 4400 0    50   Output ~ 0
+Text HLabel 8350 4000 2    50   Output ~ 0
 IO_INB
-Text HLabel 6900 4500 0    50   Output ~ 0
+Text HLabel 6900 4600 0    50   Output ~ 0
 IO_ADDR_IN
-Text HLabel 6900 4600 0    50   Output ~ 0
+Text HLabel 8350 4300 2    50   Output ~ 0
 PERIPH_MEM_SPACE
 Wire Notes Line
@@
 Text Label 2100 4200 3    50   ~ 0
 INSTR_IN
-NoConn ~ 8350 3800
-NoConn ~ 8350 3900
-NoConn ~ 8350 4000
-NoConn ~ 8350 4100
-NoConn ~ 8350 4200
-NoConn ~ 8350 4300
-NoConn ~ 8350 4400
-NoConn ~ 8350 4500
 $Comp
 L power:+3.3V #PWR?
@@
 $EndComp
 Connection ~ 2450 5650
+$Comp
+L XC9500XL:XC95144XL-10TQ100C U14
+U 6 1 5FA858A3
+P 4650 3600
+F 0 "U14" H 4650 2350 50  0000 R CNN
+F 1 "XC95144XL-10TQ100C" H 5200 2250 50  0000 R CNN
+F 2 "Package_QFP:TQFP-100_14x14mm_P0.5mm" H 4650 3600 50  0001 C CNN
+F 3 "" H 4650 3600 50  0001 C CNN
+	6    4650 3600
+	-1   0    0    -1
+$EndComp
+Text HLabel 6900 3900 0    50   Output ~ 0
+INT_OUT_I
+Text HLabel 6900 4100 0    50   Output ~ 0
+REG3_IN_L
+NoConn ~ 4350 2750
+NoConn ~ 4350 2850
+NoConn ~ 4350 2950
+NoConn ~ 4350 3050
+NoConn ~ 4350 3450
+NoConn ~ 4350 3550
+NoConn ~ 4350 3800
+NoConn ~ 4350 3900
+NoConn ~ 4350 4000
+NoConn ~ 6900 2850
+NoConn ~ 6900 2950
+NoConn ~ 6900 3050
+NoConn ~ 6900 3150
+NoConn ~ 6900 3250
+NoConn ~ 6900 3550
+NoConn ~ 6900 3650
+NoConn ~ 6900 3800
+NoConn ~ 6900 4200
+NoConn ~ 6900 4300
+NoConn ~ 6900 4400
+NoConn ~ 6900 4500
 $EndSCHEMATC
