File: pcb/homebrew-computer/registers.sch (KiCad schematic (older format))
At the start: 30 parts

Commit message: Start changing global labels with local labels
Parts:
- gave numbers to parts that had none: 25

Commit message: Start working on the pcb layout
Parts:
- C16, C17, C18, C19, C20, C21, C22, C23, C24, C25, C26, C27, C28, C29, C30, C31, C32, C33, C34, C35: footprint (none) -> Capacitor_SMD:C_0402_1005Metric_Pad0.74x0.62mm_HandSolder
- U10, U11, U12, U13, U9: footprint (none) -> Package_SO:TSSOP-48_6.1x12.5mm_P0.5mm
Connections:
- net +3V3: now reaches C16.1, C17.1, C18.1, C19.1, U9.18 (VCC), U9.31 (VCC), U9.42 (VCC), U9.7 (VCC)
- net +3V3: now also C20.1, C21.1, C22.1, C23.1, C24.1, C25.1, C26.1, C27.1, C28.1, C29.1, C30.1, C31.1, C32.1, C33.1, C34.1, C35.1, U10.18 (VCC), U10.31 (VCC), U10.42 (VCC), U10.7 (VCC), U11.18 (VCC), U11.31 (VCC), U11.42 (VCC), U11.7 (VCC), U12.18 (VCC), U12.31 (VCC), U12.42 (VCC), U12.7 (VCC), U13.18 (VCC), U13.31 (VCC), U13.42 (VCC), U13.7 (VCC)
