File: pcb/homebrew-computer/homebrew-computer.sch (KiCad schematic (older format))
At the start: 24 parts, among them J1 Conn_01x02_Male, J2 Conn_01x02_Male, J3 Conn_02x03_Counter_Clockwise, SW1 SW_Push, U1 AMS1117-3.3, U2 YC248, U3 YC248

Commit message: Keep working on the layout
Parts:
- removed U1: AMS1117-3.3, Package_TO_SOT_SMD:SOT-223-3_TabPin2, symbol Regulator_Linear:AMS1117-3.3
- added D10: LED_Small, LED_SMD:LED_0805_2012Metric, symbol Device:LED_Small
- added R8: 470, Resistor_SMD:R_0402_1005Metric_Pad0.72x0.64mm_HandSolder, symbol Device:R_Small
- added U1: TLV73333PDBV, Package_TO_SOT_SMD:SOT-23-5, symbol Regulator_Linear:TLV73333PDBV
- D1: footprint Diode_SMD:D_0603_1608Metric -> Diode_SMD:D_0603_1608Metric_Pad1.05x0.95mm_HandSolder
- D2: footprint Diode_SMD:D_0603_1608Metric -> Diode_SMD:D_0402_1005Metric_Pad0.77x0.64mm_HandSolder
- SW1: footprint Button_Switch_SMD:Panasonic_EVQPUL_EVQPUC -> Button_Switch_SMD:Panasonic_EVQPUJ_EVQPUA
Connections:
- net +3V3: now also D10.2 (A), U1.5 (OUT)
- net BUS1: now also U2.8; no longer U2.9
- net BUS10: now also U3.7; no longer U3.10
- net BUS11: now also U3.6; no longer U3.11
- net BUS12: now also U3.5; no longer U3.12
- net BUS13: now also U3.4; no longer U3.13
- net BUS14: now also U3.3; no longer U3.14
- net BUS15: now also U3.2; no longer U3.15
- net BUS16: now also U3.1; no longer U3.16
- net BUS2: now also U2.7; no longer U2.10
- net BUS3: now also U2.6; no longer U2.11
- net BUS4: now also U2.5; no longer U2.12
- net BUS5: now also U2.4; no longer U2.13
- net BUS6: now also U2.3; no longer U2.14
- net BUS7: now also U2.2; no longer U2.15
- net BUS8: now also U2.1; no longer U2.16
- net BUS9: now also U3.8; no longer U3.9
- net GND: now also U2.10, U2.11, U2.12, U2.13, U2.14, U2.15, U2.16, U2.9, U3.10, U3.11, U3.12, U3.13, U3.14, U3.15, U3.16, U3.9, R8.2, U1.2 (GND); no longer U2.1, U2.2, U2.3, U2.4, U2.5, U2.6, U2.7, U2.8, U3.1, U3.2, U3.3, U3.4, U3.5, U3.6, U3.7, U3.8
- net at C1.1, FB1.1: now also U1.1 (IN), U1.3 (EN)
- new net: D10.1 (K), R8.1
Other:
- moved on the sheet: U2, U3
Changed lines of the file:
@@
 L YC248:YC248 U?
 U 1 1 5FBC1998
-P 3550 5600
+P 3350 5600
 AR Path="/5F97DCB2/5FBC1998" Ref="U?"  Part="1"
 AR Path="/5FBC1998" Ref="U3"  Part="1"
-F 0 "U3" V 2850 5100 50  0000 L CNN
-F 1 "YC248" V 2750 5000 50  0000 L CNN
-F 2 "Resistor_SMD:YC248" H 3550 5600 50  0001 C CNN
-F 3 "" H 3550 5600 50  0001 C CNN
-	1    3550 5600
+F 0 "U3" V 2650 5000 50  0000 L CNN
+F 1 "YC248" V 2550 4900 50  0000 L CNN
+F 2 "Resistor_SMD:YC248" H 3350 5600 50  0001 C CNN
+F 3 "" H 3350 5600 50  0001 C CNN
+	1    3350 5600
 	0    -1   -1   0
 $EndComp
@@
 L YC248:YC248 U?
 U 1 1 5FBC199E
-P 3550 4350
+P 3350 4350
 AR Path="/5F97DCB2/5FBC199E" Ref="U?"  Part="1"
 AR Path="/5FBC199E" Ref="U2"  Part="1"
-F 0 "U2" V 4400 3950 50  0000 L CNN
-F 1 "YC248" V 4300 3800 50  0000 L CNN
-F 2 "Resistor_SMD:YC248" H 3550 4350 50  0001 C CNN
-F 3 "" H 3550 4350 50  0001 C CNN
-	1    3550 4350
+F 0 "U2" V 4200 3950 50  0000 L CNN
+F 1 "YC248" V 4100 3800 50  0000 L CNN
+F 2 "Resistor_SMD:YC248" H 3350 4350 50  0001 C CNN
+F 3 "" H 3350 4350 50  0001 C CNN
+	1    3350 4350
 	0    -1   -1   0
 $EndComp
@@
 L power:GND #PWR?
 U 1 1 5FBC19B4
-P 4350 6200
+P 3650 6200
 AR Path="/5F97DCB2/5FBC19B4" Ref="#PWR?"  Part="1"
 AR Path="/5FBC19B4" Ref="#PWR0121"  Part="1"
-F 0 "#PWR0121" H 4350 5950 50  0001 C CNN
-F 1 "GND" H 4355 6027 50  0000 C CNN
-F 2 "" H 4350 6200 50  0001 C CNN
-F 3 "" H 4350 6200 50  0001 C CNN
-	1    4350 6200
-	1    0    0    -1
-$EndComp
-Wire Wire Line
-	4350 6200 4350 6100
-Connection ~ 4350 3950
-Wire Wire Line
-	4350 3950 4350 3800
-Connection ~ 4350 4100
-Wire Wire Line
-	4350 4100 4350 3950
-Connection ~ 4350 4250
-Wire Wire Line
-	4350 4250 4350 4100
-Connection ~ 4350 4400
-Wire Wire Line
-	4350 4400 4350 4250
-Connection ~ 4350 4550
-Wire Wire Line
-	4350 4550 4350 4400
-Connection ~ 4350 4700
-Wire Wire Line
-	4350 4700 4350 4550
-Connection ~ 4350 4850
-Wire Wire Line
-	4350 4850 4350 4700
-Connection ~ 4350 5050
-Wire Wire Line
-	4350 5050 4350 4850
-Connection ~ 4350 5200
-Wire Wire Line
-	4350 5200 4350 5050
-Connection ~ 4350 5350
-Wire Wire Line
-	4350 5350 4350 5200
-Connection ~ 4350 5500
-Wire Wire Line
-	4350 5500 4350 5350
-Connection ~ 4350 5650
-Wire Wire Line
-	4350 5650 4350 5500
-Connection ~ 4350 5800
-Wire Wire Line
-	4350 5800 4350 5650
-Connection ~ 4350 5950
-Wire Wire Line
-	4350 5950 4350 5800
-Connection ~ 4350 6100
-Wire Wire Line
-	4350 6100 4350 5950
+F 0 "#PWR0121" H 3650 5950 50  0001 C CNN
+F 1 "GND" H 3655 6027 50  0000 C CNN
+F 2 "" H 3650 6200 50  0001 C CNN
+F 3 "" H 3650 6200 50  0001 C CNN
+	1    3650 6200
+	1    0    0    -1
+$EndComp
+Wire Wire Line
+	3650 6200 3650 6100
+Connection ~ 3650 3950
+Wire Wire Line
+	3650 3950 3650 3800
+Connection ~ 3650 4100
+Wire Wire Line
+	3650 4100 3650 3950
+Connection ~ 3650 4250
+Wire Wire Line
+	3650 4250 3650 4100
+Connection ~ 3650 4400
+Wire Wire Line
+	3650 4400 3650 4250
+Connection ~ 3650 4550
+Wire Wire Line
+	3650 4550 3650 4400
+Connection ~ 3650 4700
+Wire Wire Line
+	3650 4700 3650 4550
+Connection ~ 3650 4850
+Wire Wire Line
+	3650 4850 3650 4700
+Connection ~ 3650 5050
+Wire Wire Line
+	3650 5050 3650 4850
+Connection ~ 3650 5200
+Wire Wire Line
+	3650 5200 3650 5050
+Connection ~ 3650 5350
+Wire Wire Line
+	3650 5350 3650 5200
+Connection ~ 3650 5500
+Wire Wire Line
+	3650 5500 3650 5350
+Connection ~ 3650 5650
+Wire Wire Line
+	3650 5650 3650 5500
+Connection ~ 3650 5800
+Wire Wire Line
+	3650 5800 3650 5650
+Connection ~ 3650 5950
+Wire Wire Line
+	3650 5950 3650 5800
+Connection ~ 3650 6100
+Wire Wire Line
+	3650 6100 3650 5950
 Wire Notes Line
 	3400 6550 3400 3350
@@
 F 0 "SW1" H 1450 3785 50  0000 C CNN
 F 1 "SW_Push" H 1450 3694 50  0000 C CNN
-F 2 "Button_Switch_SMD:Panasonic_EVQPUL_EVQPUC" H 1450 3700 50  0001 C CNN
+F 2 "Button_Switch_SMD:Panasonic_EVQPUJ_EVQPUA" H 1450 3700 50  0001 C CNN
 F 3 "~" H 1450 3700 50  0001 C CNN
 	1    1450 3500
@@
 F 0 "D2" H 1850 3293 50  0000 C CNN
 F 1 "D_Small" H 1850 3384 50  0000 C CNN
-F 2 "Diode_SMD:D_0603_1608Metric" V 1850 3500 50  0001 C CNN
+F 2 "Diode_SMD:D_0402_1005Metric_Pad0.77x0.64mm_HandSolder" V 1850 3500 50  0001 C CNN
 F 3 "~" V 1850 3500 50  0001 C CNN
 	1    1850 3500
@@
 F 0 "D1" H 2000 1550 50  0000 C CNN
 F 1 "D_Schottky_Small" H 2000 1650 50  0000 C CNN
-F 2 "Diode_SMD:D_0603_1608Metric" V 2000 1800 50  0001 C CNN
+F 2 "Diode_SMD:D_0603_1608Metric_Pad1.05x0.95mm_HandSolder" V 2000 1800 50  0001 C CNN
 F 3 "~" V 2000 1800 50  0001 C CNN
 	1    2000 1800
@@
 	1    0    0    -1
 $EndComp
-Wire Wire Line
-	3300 2150 3750 2150
-Wire Wire Line
-	3750 2150 3750 2250
-Wire Wire Line
-	3750 2150 4200 2150
-Connection ~ 3750 2150
-Wire Wire Line
-	3750 2150 3750 2100
 $Comp
 L power:+3.3V #PWR02
@@
 P 4200 1800
 F 0 "#PWR02" H 4200 1650 50  0001 C CNN
-F 1 "+3.3V" H 4350 1900 50  0000 C CNN
+F 1 "+3.3V" H 4200 2000 50  0000 C CNN
 F 2 "" H 4200 1800 50  0001 C CNN
 F 3 "" H 4200 1800 50  0001 C CNN
@@
 Connection ~ 4200 1800
 Wire Notes Line
-	850  1250 4550 1250
-Wire Notes Line
-	4550 1250 4550 2550
-Wire Notes Line
-	4550 2550 850  2550
+	4800 1250 4800 2550
 Wire Notes Line
 	850  2550 850  1250
@@
 Text Label 10150 1050 0    50   ~ 0
 RESET
-Text GLabel 3850 6100 0    50   3State ~ 0
+Text GLabel 4150 6100 2    50   3State ~ 0
 BUS16
-Text GLabel 3850 5950 0    50   3State ~ 0
+Text GLabel 4150 5950 2    50   3State ~ 0
 BUS15
-Text GLabel 3850 5800 0    50   3State ~ 0
+Text GLabel 4150 5800 2    50   3State ~ 0
 BUS14
-Text GLabel 3850 5650 0    50   3State ~ 0
+Text GLabel 4150 5650 2    50   3State ~ 0
 BUS13
-Text GLabel 3850 5500 0    50   3State ~ 0
+Text GLabel 4150 5500 2    50   3State ~ 0
 BUS12
-Text GLabel 3850 5350 0    50   3State ~ 0
+Text GLabel 4150 5350 2    50   3State ~ 0
 BUS11
-Text GLabel 3850 5200 0    50   3State ~ 0
+Text GLabel 4150 5200 2    50   3State ~ 0
 BUS10
-Text GLabel 3850 5050 0    50   3State ~ 0
+Text GLabel 4150 5050 2    50   3State ~ 0
 BUS9
-Text GLabel 3850 4850 0    50   3State ~ 0
+Text GLabel 4150 4850 2    50   3State ~ 0
 BUS8
-Text GLabel 3850 4700 0    50   3State ~ 0
+Text GLabel 4150 4700 2    50   3State ~ 0
 BUS7
-Text GLabel 3850 4550 0    50   3State ~ 0
+Text GLabel 4150 4550 2    50   3State ~ 0
 BUS6
-Text GLabel 3850 4400 0    50   3State ~ 0
+Text GLabel 4150 4400 2    50   3State ~ 0
 BUS5
-Text GLabel 3850 4250 0    50   3State ~ 0
+Text GLabel 4150 4250 2    50   3State ~ 0
 BUS4
-Text GLabel 3850 4100 0    50   3State ~ 0
+Text GLabel 4150 4100 2    50   3State ~ 0
 BUS3
-Text GLabel 3850 3950 0    50   3State ~ 0
+Text GLabel 4150 3950 2    50   3State ~ 0
 BUS2
-Text GLabel 3850 3800 0    50   3State ~ 0
+Text GLabel 4150 3800 2    50   3State ~ 0
 BUS1
 Text Label 9000 5700 2    50   ~ 0
@@
 Text Label 9000 6000 2    50   ~ 0
 CTRL_TDI
-$Comp
-L Regulator_Linear:AMS1117-3.3 U1
-U 1 1 5FAE756B
-P 3750 1800
-F 0 "U1" H 3750 2042 50  0000 C CNN
-F 1 "AMS1117-3.3" H 3750 1951 50  0000 C CNN
-F 2 "Package_TO_SOT_SMD:SOT-223-3_TabPin2" H 3750 2000 50  0001 C CNN
-F 3 "http://www.advanced-monolithic.com/pdf/ds1117.pdf" H 3850 1550 50  0001 C CNN
-	1    3750 1800
-	1    0    0    -1
-$EndComp
 Connection ~ 3300 1800
 Text Label 6000 3100 0    50   ~ 0
@@
 Text Notes 3300 7050 0    50   ~ 0
 Mounting Holes
+$Comp
+L Regulator_Linear:TLV73333PDBV U1
+U 1 1 5FC11EDD
+P 3750 1900
+F 0 "U1" H 3750 2242 50  0000 C CNN
+F 1 "TLV73333PDBV" H 3750 2151 50  0000 C CNN
+F 2 "Package_TO_SOT_SMD:SOT-23-5" H 3750 2225 50  0001 C CIN
+F 3 "http://www.ti.com/lit/ds/symlink/tlv733p.pdf" H 3750 1900 50  0001 C CNN
+	1    3750 1900
+	1    0    0    -1
+$EndComp
+Wire Wire Line
+	3750 2200 3750 2250
+Wire Wire Line
+	3450 1900 3450 1800
+Connection ~ 3450 1800
+Wire Wire Line
+	3300 2150 3300 2200
+Wire Wire Line
+	3300 2200 3750 2200
+Connection ~ 3750 2200
+Wire Wire Line
+	3750 2200 4200 2200
+Wire Wire Line
+	4200 2200 4200 2150
+$Comp
+L Device:LED_Small D10
+U 1 1 5FC28711
+P 4550 1900
+F 0 "D10" V 4850 1950 50  0000 R CNN
+F 1 "LED_Small" V 4750 2100 50  0000 R CNN
+F 2 "LED_SMD:LED_0805_2012Metric" V 4550 1900 50  0001 C CNN
+F 3 "~" V 4550 1900 50  0001 C CNN
+	1    4550 1900
+	0    -1   -1   0
+$EndComp
+$Comp
+L Device:R_Small R8
+U 1 1 5FC29F1C
+P 4550 2100
+F 0 "R8" H 4609 2146 50  0000 L CNN
+F 1 "470" H 4609 2055 50  0000 L CNN
+F 2 "Resistor_SMD:R_0402_1005Metric_Pad0.72x0.64mm_HandSolder" H 4550 2100 50  0001 C CNN
+F 3 "~" H 4550 2100 50  0001 C CNN
+	1    4550 2100
+	1    0    0    -1
+$EndComp
+Wire Wire Line
+	4200 2200 4550 2200
+Connection ~ 4200 2200
+Wire Wire Line
+	4200 1800 4550 1800
+Wire Notes Line
+	850  1250 4800 1250
+Wire Notes Line
+	850  2550 4800 2550
 $EndSCHEMATC
