File: pcb/homebrew-computer/homebrew-computer.sch (KiCad schematic (older format))
At the start: 26 parts, among them J1 Conn_01x02_Male, J2 Conn_01x02_Male, J3 Conn_02x03_Counter_Clockwise, SW1 SW_Push, U1 TLV73333PDBV, U2 YC248, U3 YC248

Commit message: Keep working on the layout
Changed lines of the file:
@@
 Text Label 10150 5550 0    50   ~ 0
 PC_COUNT
+Text Label 10150 5650 0    50   ~ 0
+PC_OUT_I
 Text Label 10150 5750 0    50   ~ 0
-PC_OUT_I
-Text Label 10150 5650 0    50   ~ 0
 PC_IN
 Text Label 10150 1050 0    50   ~ 0

Commit message: Change connector for a more common one, and change the diode footprint
Parts:
- D2: footprint Diode_SMD:D_0402_1005Metric_Pad0.77x0.64mm_HandSolder -> Diode_SMD:D_0603_1608Metric_Pad1.05x0.95mm_HandSolder
Changed lines of the file:
@@
 F 0 "D2" H 1850 3293 50  0000 C CNN
 F 1 "D_Small" H 1850 3384 50  0000 C CNN
-F 2 "Diode_SMD:D_0402_1005Metric_Pad0.77x0.64mm_HandSolder" V 1850 3500 50  0001 C CNN
+F 2 "Diode_SMD:D_0603_1608Metric_Pad1.05x0.95mm_HandSolder" V 1850 3500 50  0001 C CNN
 F 3 "~" V 1850 3500 50  0001 C CNN
 	1    1850 3500
