File: pcb/homebrew-computer/io.sch (KiCad schematic (older format))
At the start: 19 parts

Commit message: Add program counter
Connections:
- net labels added: RESET
- wire segments 92 -> 91
Other:
- note added: "The interrupt controller should be reset when \nthe RESET pin is HIGH."
- note added: "This connector is slightly too small for the purpose,\nbut the next step is 50 ways."
Changed lines of the file:
@@
 	6850 2000 6850 1700
-Wire Wire Line
-	6900 2300 6850 2300
-Connection ~ 6850 2300
-Wire Wire Line
-	6850 2300 6850 2000
 Wire Wire Line
 	6900 2600 6850 2600
 Connection ~ 6850 2600
-Wire Wire Line
-	6850 2600 6850 2300
 Wire Wire Line
 	6900 2900 6850 2900
@@
 Wire Notes Line
 	750  750  4050 750
+Text HLabel 6750 2300 0    50   Input Italic 0
+RESET
+Wire Wire Line
+	6750 2300 6900 2300
+Wire Wire Line
+	6850 2000 6850 2600
+Text Notes 6300 5000 0    50   Italic 0
+This connector is slightly too small for the purpose,\nbut the next step is 50 ways.
+Text Notes 6300 5250 0    50   Italic 0
+The interrupt controller should be reset when \nthe RESET pin is HIGH.
 $EndSCHEMATC

Commit message: Start changing global labels with local labels
Parts:
- gave numbers to parts that had none: 17
Other:
- moved on the sheet: U5C

Commit message: Start working on the pcb layout
Parts:
- removed U7: 74LVC1G14GV,125, symbol 74LVC1G14:74LVC1G14GV,125
- added U7: 74LVC1G14GW,125, Package_SO:TSSOP-5, symbol 74LVC1G14:74LVC1G14GW,125
- C10, C11, C12, C7, C8, C9: footprint (none) -> Capacitor_SMD:C_0402_1005Metric_Pad0.74x0.62mm_HandSolder
- D3, D4, D5, D6, D7, D8, D9: footprint (none) -> Diode_SMD:D_0603_1608Metric
- U5: footprint (none) -> Package_SO:TSSOP-48_6.1x12.5mm_P0.5mm
- U6: footprint (none) -> Package_SO:TSSOP-16_4.4x5mm_P0.65mm
Connections:
- wire segments 91 -> 90
- no-connect marks 1 -> 2
Changed lines of the file:
@@
 $Descr User 9055 7087
 encoding utf-8
-Sheet 7 7
+Sheet 5 7
 Title "Inputs and Outputs"
 Date "2020-10-24"
@@
 F 0 "U6" H 5350 2365 50  0000 C CNN
 F 1 "SN74AVC4T245PWR" H 5350 2274 50  0000 C CNN
-F 2 "" H 5350 2300 50  0001 C CNN
+F 2 "Package_SO:TSSOP-16_4.4x5mm_P0.65mm" H 5350 2300 50  0001 C CNN
 F 3 "" H 5350 2300 50  0001 C CNN
 	1    5350 2300
@@
 F 0 "C7" H 4442 2696 50  0000 L CNN
 F 1 "100n" H 4442 2605 50  0000 L CNN
-F 2 "" H 4350 2650 50  0001 C CNN
+F 2 "Capacitor_SMD:C_0402_1005Metric_Pad0.74x0.62mm_HandSolder" H 4350 2650 50  0001 C CNN
 F 3 "~" H 4350 2650 50  0001 C CNN
 	1    4350 2650
@@
 Wire Wire Line
 	5700 2600 5700 2700
-Wire Wire Line
-	5000 3100 5000 3200
-Connection ~ 5000 3200
 NoConn ~ 5700 3100
 $Comp
@@
 F 0 "U5" H 1900 3350 50  0000 C CNN
 F 1 "SN74AVC16T245DGGR" H 1900 3300 50  0000 C CNN
-F 2 "" H 2000 3250 50  0001 C CNN
+F 2 "Package_SO:TSSOP-48_6.1x12.5mm_P0.5mm" H 2000 3250 50  0001 C CNN
 F 3 "" H 2000 3250 50  0001 C CNN
 	1    2000 3250
@@
 F 0 "U5" H 2325 4915 50  0000 C CNN
 F 1 "SN74AVC16T245DGGR" H 2325 4824 50  0000 C CNN
-F 2 "" H 2300 4900 50  0001 C CNN
+F 2 "Package_SO:TSSOP-48_6.1x12.5mm_P0.5mm" H 2300 4900 50  0001 C CNN
 F 3 "" H 2300 4900 50  0001 C CNN
 	2    2300 4900
@@
 F 0 "U5" H 2425 1015 50  0000 C CNN
 F 1 "SN74AVC16T245DGGR" H 2425 924 50  0000 C CNN
-F 2 "" H 2350 1000 50  0001 C CNN
+F 2 "Package_SO:TSSOP-48_6.1x12.5mm_P0.5mm" H 2350 1000 50  0001 C CNN
 F 3 "" H 2350 1000 50  0001 C CNN
 	3    2350 1000
@@
 F 0 "C9" H 2242 4696 50  0000 L CNN
 F 1 "100n" H 2242 4605 50  0000 L CNN
-F 2 "" H 2150 4650 50  0001 C CNN
+F 2 "Capacitor_SMD:C_0402_1005Metric_Pad0.74x0.62mm_HandSolder" H 2150 4650 50  0001 C CNN
 F 3 "~" H 2150 4650 50  0001 C CNN
 	1    2150 4650
@@
 F 0 "C10" H 2542 4696 50  0000 L CNN
 F 1 "100n" H 2542 4605 50  0000 L CNN
-F 2 "" H 2450 4650 50  0001 C CNN
+F 2 "Capacitor_SMD:C_0402_1005Metric_Pad0.74x0.62mm_HandSolder" H 2450 4650 50  0001 C CNN
 F 3 "~" H 2450 4650 50  0001 C CNN
 	1    2450 4650
@@
 F 0 "C11" H 2842 4696 50  0000 L CNN
 F 1 "100n" H 2842 4605 50  0000 L CNN
-F 2 "" H 2750 4650 50  0001 C CNN
+F 2 "Capacitor_SMD:C_0402_1005Metric_Pad0.74x0.62mm_HandSolder" H 2750 4650 50  0001 C CNN
 F 3 "~" H 2750 4650 50  0001 C CNN
 	1    2750 4650
@@
 F 0 "C8" H 1942 4696 50  0000 L CNN
 F 1 "100n" H 1942 4605 50  0000 L CNN
-F 2 "" H 1850 4650 50  0001 C CNN
+F 2 "Capacitor_SMD:C_0402_1005Metric_Pad0.74x0.62mm_HandSolder" H 1850 4650 50  0001 C CNN
 F 3 "~" H 1850 4650 50  0001 C CNN
 	1    1850 4650
@@
 F 0 "D3" H 3300 3557 50  0000 C CNN
 F 1 "D_Small" H 3500 3550 50  0000 C CNN
-F 2 "" V 3300 3350 50  0001 C CNN
+F 2 "Diode_SMD:D_0603_1608Metric" V 3300 3350 50  0001 C CNN
 F 3 "~" V 3300 3350 50  0001 C CNN
 	1    3300 3350
@@
 F 0 "D5" H 3300 3657 50  0000 C CNN
 F 1 "D_Small" H 3500 3650 50  0000 C CNN
-F 2 "" V 3300 3450 50  0001 C CNN
+F 2 "Diode_SMD:D_0603_1608Metric" V 3300 3450 50  0001 C CNN
 F 3 "~" V 3300 3450 50  0001 C CNN
 	1    3300 3450
@@
 F 0 "D7" H 3300 3050 50  0000 C CNN
 F 1 "D_Small" H 3500 3050 50  0000 C CNN
-F 2 "" V 3300 3550 50  0001 C CNN
+F 2 "Diode_SMD:D_0603_1608Metric" V 3300 3550 50  0001 C CNN
 F 3 "~" V 3300 3550 50  0001 C CNN
 	1    3300 3550
@@
 F 0 "D8" H 3300 3450 50  0000 C CNN
 F 1 "D_Small" H 3500 3450 50  0000 C CNN
-F 2 "" V 3300 3650 50  0001 C CNN
+F 2 "Diode_SMD:D_0603_1608Metric" V 3300 3650 50  0001 C CNN
 F 3 "~" V 3300 3650 50  0001 C CNN
 	1    3300 3650
@@
 F 0 "D9" H 3300 3550 50  0000 C CNN
 F 1 "D_Small" H 3500 3550 50  0000 C CNN
-F 2 "" V 3300 3750 50  0001 C CNN
+F 2 "Diode_SMD:D_0603_1608Metric" V 3300 3750 50  0001 C CNN
 F 3 "~" V 3300 3750 50  0001 C CNN
 	1    3300 3750
@@
 Wire Wire Line
 	2300 3450 2300 3500
-$Comp
-L 74LVC1G14:74LVC1G14GV,125 U?
-U 1 1 5F9B5E2D
-P 2700 3200
-AR Path="/5F95DC76/5F9B5E2D" Ref="U?"  Part="1"
-AR Path="/5F8B5DB4/5F9B5E2D" Ref="U7"  Part="1"
-F 0 "U7" H 2700 3250 50  0000 C CNN
-F 1 "74LVC1G14GV,125" H 2650 3200 50  0000 C CNN
-F 2 "" H 2700 3200 50  0001 C CNN
-F 3 "" H 2700 3200 50  0001 C CNN
-	1    2700 3200
-	-1   0    0    -1
-$EndComp
 Wire Wire Line
 	3200 3350 3200 3450
@@
 F 0 "C12" H 3192 4696 50  0000 L CNN
 F 1 "100n" H 3192 4605 50  0000 L CNN
-F 2 "" H 3100 4650 50  0001 C CNN
+F 2 "Capacitor_SMD:C_0402_1005Metric_Pad0.74x0.62mm_HandSolder" H 3100 4650 50  0001 C CNN
 F 3 "~" H 3100 4650 50  0001 C CNN
 	1    3100 4650
@@
 F 0 "D4" H 1350 3657 50  0000 C CNN
 F 1 "D_Small" H 1550 3650 50  0000 C CNN
-F 2 "" V 1350 3450 50  0001 C CNN
+F 2 "Diode_SMD:D_0603_1608Metric" V 1350 3450 50  0001 C CNN
 F 3 "~" V 1350 3450 50  0001 C CNN
 	1    1350 3450
@@
 F 0 "D6" H 1350 3757 50  0000 C CNN
 F 1 "D_Small" H 1550 3750 50  0000 C CNN
-F 2 "" V 1350 3550 50  0001 C CNN
+F 2 "Diode_SMD:D_0603_1608Metric" V 1350 3550 50  0001 C CNN
 F 3 "~" V 1350 3550 50  0001 C CNN
 	1    1350 3550
@@
 Text Label 5000 3000 2    50   ~ 0
 INT2
+NoConn ~ 5000 3100
+$Comp
+L 74LVC1G14:74LVC1G14GW,125 U7
+U 1 1 5FADD492
+P 2700 3200
+F 0 "U7" H 2675 3265 50  0000 C CNN
+F 1 "74LVC1G14GW,125" H 2675 3174 50  0000 C CNN
+F 2 "Package_SO:TSSOP-5" H 2700 3200 50  0001 C CNN
+F 3 "" H 2700 3200 50  0001 C CNN
+	1    2700 3200
+	-1   0    0    -1
+$EndComp
 $EndSCHEMATC

Commit message: Keep working on the layout
Parts:
- removed J4: Conn_02x20_Counter_Clockwise, symbol Connector_Generic:Conn_02x20_Counter_Clockwise
- added J4: Conn_02x20_Odd_Even, Connector_Molex:Molex_Pico-Clasp_203566-4007_2x20_P1.00mm_Horizontal, symbol Connector_Generic:Conn_02x20_Odd_Even
Connections:
- net GND: now also J4.1 (Pin_1), J4.13 (Pin_13), J4.14 (Pin_14), J4.19 (Pin_19), J4.2 (Pin_2), J4.20 (Pin_20), J4.26 (Pin_26), J4.31 (Pin_31), J4.32 (Pin_32), J4.37 (Pin_37), J4.7 (Pin_7), J4.8 (Pin_8)
- net INT: now also J4.27 (Pin_27)
- net INT0: now also J4.29 (Pin_29)
- net INT1: now also J4.33 (Pin_33)
- net INT2: now also J4.35 (Pin_35)
- net IO1: now also J4.3 (Pin_3)
- net IO10: now also J4.24 (Pin_24)
- net IO11: now also J4.16 (Pin_16)
- net IO12: now also J4.18 (Pin_18)
- net IO13: now also J4.10 (Pin_10)
- net IO14: now also J4.12 (Pin_12)
- net IO15: now also J4.4 (Pin_4)
- net IO16: now also J4.6 (Pin_6)
- net IO2: now also J4.5 (Pin_5)
- net IO3: now also J4.9 (Pin_9)
- net IO4: now also J4.11 (Pin_11)
- net IO5: now also J4.15 (Pin_15)
- net IO6: now also J4.17 (Pin_17)
- net IO7: now also J4.21 (Pin_21)
- net IO8: now also J4.23 (Pin_23)
- net IO9: now also J4.22 (Pin_22)
- net IO_ADDR_IN: now also J4.28 (Pin_28)
- net IO_IN: now also J4.34 (Pin_34)
- net IO_INB: now also J4.38 (Pin_38)
- net IO_OUT: now also J4.30 (Pin_30)
- net IO_OUTB: now also J4.36 (Pin_36)
- net PERIPH_MEM_SPACE: now also J4.40 (Pin_40)
- net RESET: now also J4.25 (Pin_25)
- net RST_INT: now also J4.39 (Pin_39)
Changed lines of the file:
@@
 Text Notes 6300 4050 0    50   Italic 0
 The clock is not sent through this connector.\nIt is passed by another connector to the clock module,\nin the external clock configuration
-$Comp
-L Connector_Generic:Conn_02x20_Counter_Clockwise J4
-U 1 1 5F93FA7B
-P 7100 2000
-F 0 "J4" H 7150 3117 50  0000 C CNN
-F 1 "Conn_02x20_Counter_Clockwise" H 7150 3026 50  0000 C CNN
-F 2 "" H 7100 2000 50  0001 C CNN
-F 3 "~" H 7100 2000 50  0001 C CNN
-	1    7100 2000
-	1    0    0    -1
-$EndComp
 Text Notes 6300 4400 0    50   Italic 0
 We need to care about ground return path.\nIt doesn’t have to be perfect, but we should\ninclude at least a few ground connections
@@
 	-1   0    0    -1
 $EndComp
+$Comp
+L Connector_Generic:Conn_02x20_Odd_Even J4
+U 1 1 5FAD2DAF
+P 7100 2000
+F 0 "J4" H 7150 3117 50  0000 C CNN
+F 1 "Conn_02x20_Odd_Even" H 7150 3026 50  0000 C CNN
+F 2 "Connector_Molex:Molex_Pico-Clasp_203566-4007_2x20_P1.00mm_Horizontal" H 7100 2000 50  0001 C CNN
+F 3 "~" H 7100 2000 50  0001 C CNN
+	1    7100 2000
+	1    0    0    -1
+$EndComp
 $EndSCHEMATC

Commit message: Add the board outline
Parts:
- U7: footprint Package_SO:TSSOP-5 -> Package_TO_SOT_SMD:SOT-353_SC-70-5_Handsoldering
Changed lines of the file:
@@
 F 0 "U7" H 2675 3265 50  0000 C CNN
 F 1 "74LVC1G14GW,125" H 2675 3174 50  0000 C CNN
-F 2 "Package_SO:TSSOP-5" H 2700 3200 50  0001 C CNN
+F 2 "Package_TO_SOT_SMD:SOT-353_SC-70-5_Handsoldering" H 2700 3200 50  0001 C CNN
 F 3 "" H 2700 3200 50  0001 C CNN
 	1    2700 3200

Commit message: Keep working on the layout
Parts:
- D3, D4, D5, D6, D7, D8, D9: footprint Diode_SMD:D_0603_1608Metric -> Diode_SMD:D_0402_1005Metric_Pad0.77x0.64mm_HandSolder
- U7: footprint Package_TO_SOT_SMD:SOT-353_SC-70-5_Handsoldering -> Package_TO_SOT_SMD:SOT-353_SC-70-5
Connections:
- net +3V3: no longer D4.1 (K), D6.1 (K), U5.1 (1DIR), U5.24 (2DIR)
- net GND: now also J4.11 (Pin_11), J4.12 (Pin_12), J4.17 (Pin_17), J4.18 (Pin_18), J4.23 (Pin_23), J4.24 (Pin_24), J4.29 (Pin_29), J4.30 (Pin_30), J4.35 (Pin_35), J4.36 (Pin_36), J4.5 (Pin_5), J4.6 (Pin_6); no longer J4.1 (Pin_1), J4.13 (Pin_13), J4.14 (Pin_14), J4.19 (Pin_19), J4.2 (Pin_2), J4.20 (Pin_20), J4.26 (Pin_26), J4.31 (Pin_31), J4.32 (Pin_32), J4.37 (Pin_37), J4.7 (Pin_7), J4.8 (Pin_8)
- net INT: now also J4.2 (Pin_2); no longer J4.27 (Pin_27)
- net INT0: now also J4.4 (Pin_4); no longer J4.29 (Pin_29)
- net INT1: now also J4.8 (Pin_8); no longer J4.33 (Pin_33)
- net INT2: now also J4.10 (Pin_10); no longer J4.35 (Pin_35)
- net IO1: now also J4.1 (Pin_1); no longer J4.3 (Pin_3)
- net IO10: now also J4.27 (Pin_27); no longer J4.24 (Pin_24)
- net IO11: now also J4.31 (Pin_31); no longer J4.16 (Pin_16)
- net IO12: now also J4.33 (Pin_33); no longer J4.18 (Pin_18)
- net IO13: now also J4.37 (Pin_37); no longer J4.10 (Pin_10)
- net IO14: now also J4.39 (Pin_39); no longer J4.12 (Pin_12)
- net IO15: now also J4.38 (Pin_38); no longer J4.4 (Pin_4)
- net IO16: now also J4.40 (Pin_40); no longer J4.6 (Pin_6)
- net IO2: now also J4.3 (Pin_3); no longer J4.5 (Pin_5)
- net IO3: now also J4.7 (Pin_7); no longer J4.9 (Pin_9)
- net IO4: now also J4.9 (Pin_9); no longer J4.11 (Pin_11)
- net IO5: now also J4.13 (Pin_13); no longer J4.15 (Pin_15)
- net IO6: now also J4.15 (Pin_15); no longer J4.17 (Pin_17)
- net IO7: now also J4.19 (Pin_19); no longer J4.21 (Pin_21)
- net IO8: now also J4.21 (Pin_21); no longer J4.23 (Pin_23)
- net IO9: now also J4.25 (Pin_25); no longer J4.22 (Pin_22)
- net IO_ADDR_IN: now also J4.20 (Pin_20); no longer J4.28 (Pin_28)
- net IO_IN: now also J4.26 (Pin_26); no longer J4.34 (Pin_34)
- net IO_INB: now also J4.32 (Pin_32); no longer J4.38 (Pin_38)
- net IO_OUT: now also J4.22 (Pin_22); no longer J4.30 (Pin_30)
- net IO_OUTB: now also J4.28 (Pin_28); no longer J4.36 (Pin_36)
- net PERIPH_MEM_SPACE: now also J4.34 (Pin_34); no longer J4.40 (Pin_40)
- net RESET: now also J4.16 (Pin_16); no longer J4.25 (Pin_25)
- net RST_INT: now also J4.14 (Pin_14); no longer J4.39 (Pin_39)
- new net: D4.1 (K), D6.1 (K), U5.1 (1DIR), U5.24 (2DIR)

Commit message: Keep working on the layout
Connections:
- net INT0: now also J4.10 (Pin_10); no longer J4.4 (Pin_4)
- net INT2: now also J4.4 (Pin_4); no longer J4.10 (Pin_10)
Changed lines of the file:
@@
 Text Label 7550 3000 0    50   ~ 0
 IO16
-Text Label 7550 1200 0    50   ~ 0
+Text Label 7550 1500 0    50   ~ 0
 INT0
 Text Label 7550 1400 0    50   ~ 0
 INT1
-Text Label 7550 1500 0    50   ~ 0
+Text Label 7550 1200 0    50   ~ 0
 INT2
 Text Label 5000 2800 2    50   ~ 0
