File: pcb/homebrew-computer/io.sch (KiCad schematic (older format))
At the start: 17 parts, among them J4 Conn_02x20_Odd_Even, U5 SN74AVC16T245DGGR, U6 SN74AVC4T245PWR, U7 74LVC1G14GW,125

Commit message: Finished working on the layout
Connections:
- net INT: now also J4.26 (Pin_26); no longer J4.2 (Pin_2)
- net INT0: now also J4.8 (Pin_8); no longer J4.10 (Pin_10)
- net INT1: now also J4.4 (Pin_4); no longer J4.8 (Pin_8)
- net INT2: now also J4.2 (Pin_2); no longer J4.4 (Pin_4)
- net IO_ADDR_IN: now also J4.10 (Pin_10); no longer J4.20 (Pin_20)
- net IO_IN: now also J4.16 (Pin_16); no longer J4.26 (Pin_26)
- net IO_INB: now also J4.22 (Pin_22); no longer J4.32 (Pin_32)
- net IO_OUT: now also J4.14 (Pin_14); no longer J4.22 (Pin_22)
- net IO_OUTB: now also J4.20 (Pin_20); no longer J4.28 (Pin_28)
- net PERIPH_MEM_SPACE: now also J4.32 (Pin_32); no longer J4.34 (Pin_34)
- net RESET: now also J4.34 (Pin_34); no longer J4.16 (Pin_16)
- net RST_INT: now also J4.28 (Pin_28); no longer J4.14 (Pin_14)
Changed lines of the file:
@@
 Text Notes 6300 750  0    50   ~ 0
 IO connector
-Text HLabel 7550 1100 2    50   Output ~ 0
-INT
 $Comp
 L 74AVC4T245:SN74AVC4T245PWR U6
@@
 Wire Notes Line
 	4150 3650 6150 3650
-Text HLabel 7550 1700 2    50   Input Italic 0
-RST_INT
 Wire Wire Line
 	7400 2400 7550 2400
@@
 Wire Notes Line
 	4050 6450 4050 750
-Text HLabel 7550 2700 2    50   Input ~ 0
-PERIPH_MEM_SPACE
 Wire Wire Line
 	7400 2900 7550 2900
@@
 Wire Notes Line
 	6300 3400 8400 3400
-Text HLabel 7550 2000 2    50   Input ~ 0
-IO_ADDR_IN
-Text HLabel 7550 2100 2    50   Input ~ 0
-IO_OUT
-Text HLabel 7550 2300 2    50   Input ~ 0
-IO_IN
-Text HLabel 7550 2400 2    50   Input ~ 0
-IO_OUTB
-Text HLabel 7550 2600 2    50   Input ~ 0
-IO_INB
 Text Notes 850  4150 0    50   Italic 0
 We use diodes to implement the OR\nfunction as there will only be one \nactive at the same time
@@
 Wire Notes Line
 	750  750  4050 750
-Text HLabel 7550 1800 2    50   Input Italic 0
-RESET
 Wire Wire Line
 	6750 2300 6900 2300
@@
 Text Label 7550 3000 0    50   ~ 0
 IO16
-Text Label 7550 1500 0    50   ~ 0
-INT0
-Text Label 7550 1400 0    50   ~ 0
-INT1
-Text Label 7550 1200 0    50   ~ 0
-INT2
 Text Label 5000 2800 2    50   ~ 0
 INT0
@@
 Wire Wire Line
 	7450 2500 7450 2800
+Text HLabel 7550 2600 2    50   Input ~ 0
+PERIPH_MEM_SPACE
+Text HLabel 7550 2100 2    50   Input ~ 0
+IO_INB
+Text HLabel 7550 2000 2    50   Input ~ 0
+IO_OUTB
+Text HLabel 7550 1800 2    50   Input ~ 0
+IO_IN
+Text HLabel 7550 1700 2    50   Input ~ 0
+IO_OUT
+Text HLabel 7550 1500 2    50   Input ~ 0
+IO_ADDR_IN
+Text Label 7550 1100 0    50   ~ 0
+INT2
+Text Label 7550 1200 0    50   ~ 0
+INT1
+Text Label 7550 1400 0    50   ~ 0
+INT0
+Text HLabel 7550 2700 2    50   Input Italic 0
+RESET
+Text HLabel 7550 2400 2    50   Input Italic 0
+RST_INT
+Text HLabel 7550 2300 2    50   Output ~ 0
+INT
 $EndSCHEMATC

Commit message: Change connector for a more common one, and change the diode footprint
Parts:
- D3, D4, D5, D6, D7, D8, D9: footprint Diode_SMD:D_0402_1005Metric_Pad0.77x0.64mm_HandSolder -> Diode_SMD:D_0603_1608Metric_Pad1.05x0.95mm_HandSolder
- J4: footprint Connector_Molex:Molex_Pico-Clasp_203566-4007_2x20_P1.00mm_Horizontal -> Connector_Molex:Micro-Lock-Plus-02x20
Changed lines of the file:
@@
 F 0 "D3" H 3300 3557 50  0000 C CNN
 F 1 "D_Small" H 3500 3550 50  0000 C CNN
-F 2 "Diode_SMD:D_0402_1005Metric_Pad0.77x0.64mm_HandSolder" V 3300 3350 50  0001 C CNN
+F 2 "Diode_SMD:D_0603_1608Metric_Pad1.05x0.95mm_HandSolder" V 3300 3350 50  0001 C CNN
 F 3 "~" V 3300 3350 50  0001 C CNN
 	1    3300 3350
@@
 F 0 "D5" H 3300 3657 50  0000 C CNN
 F 1 "D_Small" H 3500 3650 50  0000 C CNN
-F 2 "Diode_SMD:D_0402_1005Metric_Pad0.77x0.64mm_HandSolder" V 3300 3450 50  0001 C CNN
+F 2 "Diode_SMD:D_0603_1608Metric_Pad1.05x0.95mm_HandSolder" V 3300 3450 50  0001 C CNN
 F 3 "~" V 3300 3450 50  0001 C CNN
 	1    3300 3450
@@
 F 0 "D7" H 3300 3050 50  0000 C CNN
 F 1 "D_Small" H 3500 3050 50  0000 C CNN
-F 2 "Diode_SMD:D_0402_1005Metric_Pad0.77x0.64mm_HandSolder" V 3300 3550 50  0001 C CNN
+F 2 "Diode_SMD:D_0603_1608Metric_Pad1.05x0.95mm_HandSolder" V 3300 3550 50  0001 C CNN
 F 3 "~" V 3300 3550 50  0001 C CNN
 	1    3300 3550
@@
 F 0 "D8" H 3300 3450 50  0000 C CNN
 F 1 "D_Small" H 3500 3450 50  0000 C CNN
-F 2 "Diode_SMD:D_0402_1005Metric_Pad0.77x0.64mm_HandSolder" V 3300 3650 50  0001 C CNN
+F 2 "Diode_SMD:D_0603_1608Metric_Pad1.05x0.95mm_HandSolder" V 3300 3650 50  0001 C CNN
 F 3 "~" V 3300 3650 50  0001 C CNN
 	1    3300 3650
@@
 F 0 "D9" H 3300 3550 50  0000 C CNN
 F 1 "D_Small" H 3500 3550 50  0000 C CNN
-F 2 "Diode_SMD:D_0402_1005Metric_Pad0.77x0.64mm_HandSolder" V 3300 3750 50  0001 C CNN
+F 2 "Diode_SMD:D_0603_1608Metric_Pad1.05x0.95mm_HandSolder" V 3300 3750 50  0001 C CNN
 F 3 "~" V 3300 3750 50  0001 C CNN
 	1    3300 3750
@@
 F 0 "D4" H 1350 3657 50  0000 C CNN
 F 1 "D_Small" H 1550 3650 50  0000 C CNN
-F 2 "Diode_SMD:D_0402_1005Metric_Pad0.77x0.64mm_HandSolder" V 1350 3450 50  0001 C CNN
+F 2 "Diode_SMD:D_0603_1608Metric_Pad1.05x0.95mm_HandSolder" V 1350 3450 50  0001 C CNN
 F 3 "~" V 1350 3450 50  0001 C CNN
 	1    1350 3450
@@
 F 0 "D6" H 1350 3757 50  0000 C CNN
 F 1 "D_Small" H 1550 3750 50  0000 C CNN
-F 2 "Diode_SMD:D_0402_1005Metric_Pad0.77x0.64mm_HandSolder" V 1350 3550 50  0001 C CNN
+F 2 "Diode_SMD:D_0603_1608Metric_Pad1.05x0.95mm_HandSolder" V 1350 3550 50  0001 C CNN
 F 3 "~" V 1350 3550 50  0001 C CNN
 	1    1350 3550
@@
 F 0 "J4" H 7150 3117 50  0000 C CNN
 F 1 "Conn_02x20_Odd_Even" H 7150 3026 50  0000 C CNN
-F 2 "Connector_Molex:Molex_Pico-Clasp_203566-4007_2x20_P1.00mm_Horizontal" H 7100 2000 50  0001 C CNN
+F 2 "Connector_Molex:Micro-Lock-Plus-02x20" H 7100 2000 50  0001 C CNN
 F 3 "~" H 7100 2000 50  0001 C CNN
 	1    7100 2000
