File: pcb/homebrew-computer/homebrew-computer.kicad_pcb (KiCad board)
At the start: 4 copper layers, 100 x 50 mm, 100 parts, among them J1 Conn_01x02_Male, J2 Conn_01x02_Male, J3 Conn_02x03_Counter_Clockwise, J4 Conn_02x20_Odd_Even, J5 Conn_01x04_Male, J6 Conn_01x02, SW1 SW_Push, U1 TLV73333PDBV, U10 74LVC16374ADGG,112, U11 74LVC16374ADGG,112, U12 74LVC16374ADGG,112, U13 74LVC16374ADGG,112, U14 XC95144XL-10TQ100C, U15 74LVC16374ADGG,112, U16 DS1077LZ-60+, U17 74LVC1G157GC-Q100H, U18 74LVC1G14GW,125, U2 YC248, U3 YC248, U4 XC9572XL-10VQG44C, U5 SN74AVC16T245DGGR, U6 SN74AVC4T245PWR, U7 74LVC1G14GW,125, U8 XC9536XL-10VQG44C, U9 74LVC16374ADGG,112

Commit message: Keep working on the layout
Connections:
- U14 pad 1: /Control Logic/IR8 -> /Control Logic/IR7
- U14 pad 10: /Control Logic/IR16 -> /Control Logic/IR15
- U14 pad 11: /REG3_IN_L -> /Control Logic/IR16
- U14 pad 14: /ALU_OUT_I -> Net-(U14-Pad14)
- U14 pad 2: /Control Logic/IR9 -> /Control Logic/IR8
- U14 pad 3: /Control Logic/IR10 -> /Control Logic/IR9
- U14 pad 4: /Control Logic/IR11 -> /Control Logic/IR10
- U14 pad 6: /Control Logic/IR12 -> /Control Logic/IR11
- U14 pad 7: /Control Logic/IR13 -> /Control Logic/IR12
- U14 pad 8: /Control Logic/IR14 -> /Control Logic/IR13
- U14 pad 9: /Control Logic/IR15 -> /Control Logic/IR14
- U14 pad 90: /Control Logic/IR1 -> /ALU_OUT_I
- U14 pad 91: /Control Logic/IR2 -> /Control Logic/IR1
- U14 pad 92: /Control Logic/IR3 -> /Control Logic/IR2
- U14 pad 93: /Control Logic/IR4 -> /Control Logic/IR3
- U14 pad 94: /Control Logic/IR5 -> /Control Logic/IR4
- U14 pad 95: /Control Logic/IR6 -> /Control Logic/IR5
- U14 pad 96: /Control Logic/IR7 -> /Control Logic/IR6
Routing:
- net /ALU_OUT_I: track 0.00 -> 39.4 mm, vias 0 -> 1
- net /SP_OUT_I: track 24.1 -> 35.9 mm
- net /SP_IN: track 16.5 -> 28.3 mm
- net /BP_OUT_I: track 15.4 -> 27.2 mm
- net /BP_IN: track 23.9 -> 35.7 mm
- net /Control Logic/IR7: track 17.8 -> 21.0 mm
- net /Control Logic/IR8: track 21.0 -> 22.7 mm
- net /Control Logic/IR11: track 24.9 -> 26.1 mm
- net /A_IN: track 30.8 -> 31.6 mm
- net /Control Logic/IR15: track 29.8 -> 30.5 mm
- net /Control Logic/IR16: track 30.8 -> 31.5 mm
- net /Control Logic/IR14: track 28.3 -> 29.0 mm
- net /Control Logic/IR10: track 23.6 -> 24.3 mm
- net /Control Logic/IR12: track 26.2 -> 26.9 mm
- net /Control Logic/IR13: track 27.5 -> 28.2 mm
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
Commit message: Finished working on the layout
Parts:
- moved D5 7.31 mm to (100.6, 89.1), turned to 270 degrees
- moved C12 7.13 mm to (118.3, 86.2), turned to 0 degrees
- moved D8 6.98 mm to (101.9, 89.1), turned to 270 degrees
- moved D6 6.91 mm to (99.3, 89.1), turned to 270 degrees
- moved D9 6.74 mm to (94.1, 89.1), turned to 270 degrees
- moved C7 5.95 mm to (107.0, 86.7), turned to 90 degrees
- moved D4 5.31 mm to (96.7, 89.1), turned to 270 degrees
- moved C10 5.25 mm to (113.7, 91.8), turned to 180 degrees
- moved U7 4.59 mm to (118.8, 88.6), turned to 180 degrees
- moved D7 4.27 mm to (98.0, 89.1), turned to 270 degrees
- moved D3 2.57 mm to (95.4, 89.1), turned to 270 degrees
- moved C14 0.71 mm to (116.7, 95.8), turned to 315 degrees
- moved C32 0.55 mm to (101.2, 97.8)
- moved C9 0.40 mm to (118.5, 97.8)
- moved C44 0.25 mm to (87.8, 111.8)
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Connections:
- J4 pad 10: /IO/INT0 -> /IO_ADDR_IN
- J4 pad 14: /RST_INT -> /IO_OUT
- J4 pad 16: /RESET -> /IO_IN
- J4 pad 2: /INT -> /IO/INT2
- J4 pad 20: /IO_ADDR_IN -> /IO_OUTB
- J4 pad 22: /IO_OUT -> /IO_INB
- J4 pad 26: /IO_IN -> /INT
- J4 pad 28: /IO_OUTB -> /RST_INT
- J4 pad 32: /IO_INB -> /PERIPH_MEM_SPACE
- J4 pad 34: /PERIPH_MEM_SPACE -> /RESET
- J4 pad 4: /IO/INT2 -> /IO/INT1
- J4 pad 8: /IO/INT1 -> /IO/INT0
- U14 pad 16: Net-(U14-Pad16) -> /REG1_OUT_L_I
- U14 pad 17: Net-(U14-Pad17) -> /REG1_IN_L
- U14 pad 18: Net-(U14-Pad18) -> /REG1_OUT_H_I
- U14 pad 35: Net-(U14-Pad35) -> /REG2_IN_H
- U14 pad 41: /REG3_IN_H -> Net-(U14-Pad41)
- U14 pad 42: Net-(U14-Pad42) -> /REG2_OUT_L_I
- U14 pad 43: Net-(U14-Pad43) -> /REG2_IN_L
- U14 pad 50: /INT -> Net-(U14-Pad50)
- U14 pad 53: /RST_INT -> /REG3_OUT_L_I
- U14 pad 54: /IO_OUT -> /REG3_IN_L
- U14 pad 55: /IO_IN -> Net-(U14-Pad55)
- U14 pad 56: /IO_OUTB -> Net-(U14-Pad56)
- U14 pad 58: /IO_INB -> Net-(U14-Pad58)
- U14 pad 59: /IO_ADDR_IN -> Net-(U14-Pad59)
- U14 pad 60: /PERIPH_MEM_SPACE -> /IO_ADDR_IN
- U14 pad 61: Net-(U14-Pad61) -> /IO_OUT
- U14 pad 63: Net-(U14-Pad63) -> /IO_IN
- U14 pad 64: Net-(U14-Pad64) -> /IO_OUTB
- U14 pad 65: Net-(U14-Pad65) -> /IO_INB
- U14 pad 66: Net-(U14-Pad66) -> /INT
- U14 pad 67: Net-(U14-Pad67) -> /RST_INT
- U14 pad 68: Net-(U14-Pad68) -> /PERIPH_MEM_SPACE
- U14 pad 70: Net-(U14-Pad70) -> /REG3_OUT_H_I
- U14 pad 71: Net-(U14-Pad71) -> /REG3_IN_H
Routing:
- net GND: track 0.00 -> 162.3 mm, vias 0 -> 153
- net /RESET: track 11.1 -> 162.1 mm, vias 1 -> 3
- net +3V3: track 2.56 -> 146.5 mm, vias 0 -> 70
- net /IO_OUTB: track 0.00 -> 54.5 mm
- net /IO_OUT: track 0.00 -> 53.8 mm
- net /IO_ADDR_IN: track 0.00 -> 53.2 mm
- net /TMS: track 2.11 -> 54.8 mm, vias 1 -> 4
- net /IO_IN: track 0.00 -> 52.4 mm
- net /ALU_TDI: track 2.11 -> 54.1 mm, vias 1 -> 2
- net /IO_INB: track 0.00 -> 50.8 mm
- net /TCK: track 0.00 -> 49.2 mm, vias 0 -> 4
- net /PERIPH_MEM_SPACE: track 0.00 -> 48.7 mm
- net /INT: track 0.00 -> 48.2 mm
- net /RST_INT: track 0.00 -> 48.2 mm
- net /CTRL_TDI: track 0.00 -> 40.6 mm
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
Commit message: Add via stiching
Routing:
- net GND: vias 153 -> 245
Changed lines of the file:
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@@
     (thickness 1.6)
     (drawings 4)
-    (tracks 1916)
+    (tracks 2008)
     (zones 0)
     (modules 100)
@@
   (segment (start 114.975 93.75) (end 114.55 94.175) (width 0.3) (layer F.Cu) (net 2))
   (segment (start 91.75 105.3) (end 91.75 104.75) (width 0.3) (layer B.Cu) (net 2))
+  (via (at 40 95) (size 0.6) (drill 0.3) (layers F.Cu B.Cu) (net 2))
+  (via (at 40 100) (size 0.6) (drill 0.3) (layers F.Cu B.Cu) (net 2))
+  (via (at 40 105) (size 0.6) (drill 0.3) (layers F.Cu B.Cu) (net 2))
+  (via (at 40 110) (size 0.6) (drill 0.3) (layers F.Cu B.Cu) (net 2))
+  (via (at 40 115) (size 0.6) (drill 0.3) (layers F.Cu B.Cu) (net 2))
+  (via (at 40 120) (size 0.6) (drill 0.3) (layers F.Cu B.Cu) (net 2))
+  (via (at 45 120) (size 0.6) (drill 0.3) (layers F.Cu B.Cu) (net 2))
+  (via (at 45 125) (size 0.6) (drill 0.3) (layers F.Cu B.Cu) (net 2))
+  (via (at 45 115) (size 0.6) (drill 0.3) (layers F.Cu B.Cu) (net 2))
+  (via (at 45 110) (size 0.6) (drill 0.3) (layers F.Cu B.Cu) (net 2))
+  (via (at 45 105) (size 0.6) (drill 0.3) (layers F.Cu B.Cu) (net 2))
+  (via (at 45 100) (size 0.6) (drill 0.3) (layers F.Cu B.Cu) (net 2))
+  (via (at 45 95) (size 0.6) (drill 0.3) (layers F.Cu B.Cu) (net 2))
+  (via (at 45 90) (size 0.6) (drill 0.3) (layers F.Cu B.Cu) (net 2))
+  (via (at 50 80) (size 0.6) (drill 0.3) (layers F.Cu B.Cu) (net 2))
+  (via (at 50 85) (size 0.6) (drill 0.3) (layers F.Cu B.Cu) (net 2))
+  (via (at 50 90) (size 0.6) (drill 0.3) (layers F.Cu B.Cu) (net 2))
+  (via (at 50 95) (size 0.6) (drill 0.3) (layers F.Cu B.Cu) (net 2))
+  (via (at 50 100) (size 0.6) (drill 0.3) (layers F.Cu B.Cu) (net 2))
+  (via (at 50 105) (size 0.6) (drill 0.3) (layers F.Cu B.Cu) (net 2))
+  (via (at 50 110) (size 0.6) (drill 0.3) (layers F.Cu B.Cu) (net 2))
+  (via (at 50 115) (size 0.6) (drill 0.3) (layers F.Cu B.Cu) (net 2))
+  (via (at 50 120) (size 0.6) (drill 0.3) (layers F.Cu B.Cu) (net 2))
+  (via (at 50 125) (size 0.6) (drill 0.3) (layers F.Cu B.Cu) (net 2))
+  (via (at 55 120) (size 0.6) (drill 0.3) (layers F.Cu B.Cu) (net 2))
+  (via (at 55 115) (size 0.6) (drill 0.3) (layers F.Cu B.Cu) (net 2))
+  (via (at 55 90) (size 0.6) (drill 0.3) (layers F.Cu B.Cu) (net 2))
+  (via (at 55 85) (size 0.6) (drill 0.3) (layers F.Cu B.Cu) (net 2))
+  (via (at 60 85) (size 0.6) (drill 0.3) (layers F.Cu B.Cu) (net 2))
+  (via (at 65 80) (size 0.6) (drill 0.3) (layers F.Cu B.Cu) (net 2))
+  (via (at 65 85) (size 0.6) (drill 0.3) (layers F.Cu B.Cu) (net 2))
+  (via (at 60 115) (size 0.6) (drill 0.3) (layers F.Cu B.Cu) (net 2))
+  (via (at 65 125) (size 0.6) (drill 0.3) (layers F.Cu B.Cu) (net 2))
+  (via (at 70 125) (size 0.6) (drill 0.3) (layers F.Cu B.Cu) (net 2))
+  (via (at 70 120) (size 0.6) (drill 0.3) (layers F.Cu B.Cu) (net 2))
+  (via (at 70 115) (size 0.6) (drill 0.3) (layers F.Cu B.Cu) (net 2))
+  (via (at 70 85) (size 0.6) (drill 0.3) (layers F.Cu B.Cu) (net 2))
+  (via (at 70 80) (size 0.6) (drill 0.3) (layers F.Cu B.Cu) (net 2))
+  (via (at 75 80) (size 0.6) (drill 0.3) (layers F.Cu B.Cu) (net 2))
+  (via (at 75 85) (size 0.6) (drill 0.3) (layers F.Cu B.Cu) (net 2))
+  (via (at 75 115) (size 0.6) (drill 0.3) (layers F.Cu B.Cu) (net 2))
+  (via (at 75 125) (size 0.6) (drill 0.3) (layers F.Cu B.Cu) (net 2))
+  (via (at 80 125) (size 0.6) (drill 0.3) (layers F.Cu B.Cu) (net 2))
+  (via (at 80 115) (size 0.6) (drill 0.3) (layers F.Cu B.Cu) (net 2))
+  (via (at 80 85) (size 0.6) (drill 0.3) (layers F.Cu B.Cu) (net 2))
+  (via (at 80 80) (size 0.6) (drill 0.3) (layers F.Cu B.Cu) (net 2))
+  (via (at 85 80) (size 0.6) (drill 0.3) (layers F.Cu B.Cu) (net 2))
+  (via (at 85 85) (size 0.6) (drill 0.3) (layers F.Cu B.Cu) (net 2))
+  (via (at 95 80) (size 0.6) (drill 0.3) (layers F.Cu B.Cu) (net 2))
+  (via (at 95 85) (size 0.6) (drill 0.3) (layers F.Cu B.Cu) (net 2))
+  (via (at 90 85) (size 0.6) (drill 0.3) (layers F.Cu B.Cu) (net 2))
+  (via (at 100 85) (size 0.6) (drill 0.3) (layers F.Cu B.Cu) (net 2))
+  (via (at 100 80) (size 0.6) (drill 0.3) (layers F.Cu B.Cu) (net 2))
+  (via (at 100 80) (size 0.6) (drill 0.3) (layers F.Cu B.Cu) (net 2))
+  (via (at 105 85) (size 0.6) (drill 0.3) (layers F.Cu B.Cu) (net 2))
+  (via (at 105 80) (size 0.6) (drill 0.3) (layers F.Cu B.Cu) (net 2))
+  (via (at 110 80) (size 0.6) (drill 0.3) (layers F.Cu B.Cu) (net 2))
+  (via (at 115 80) (size 0.6) (drill 0.3) (layers F.Cu B.Cu) (net 2))
+  (via (at 120 80) (size 0.6) (drill 0.3) (layers F.Cu B.Cu) (net 2))
+  (via (at 125 85) (size 0.6) (drill 0.3) (layers F.Cu B.Cu) (net 2))
+  (via (at 125 80) (size 0.6) (drill 0.3) (layers F.Cu B.Cu) (net 2))
+  (via (at 130 80) (size 0.6) (drill 0.3) (layers F.Cu B.Cu) (net 2))
+  (via (at 130 85) (size 0.6) (drill 0.3) (layers F.Cu B.Cu) (net 2))
+  (via (at 135 85) (size 0.6) (drill 0.3) (layers F.Cu B.Cu) (net 2))
+  (via (at 130 90) (size 0.6) (drill 0.3) (layers F.Cu B.Cu) (net 2))
+  (via (at 135 90) (size 0.6) (drill 0.3) (layers F.Cu B.Cu) (net 2))
+  (via (at 135 115) (size 0.6) (drill 0.3) (layers F.Cu B.Cu) (net 2))
+  (via (at 130 115) (size 0.6) (drill 0.3) (layers F.Cu B.Cu) (net 2))
+  (via (at 130 120) (size 0.6) (drill 0.3) (layers F.Cu B.Cu) (net 2))
+  (via (at 135 120) (size 0.6) (drill 0.3) (layers F.Cu B.Cu) (net 2))
+  (via (at 130 125) (size 0.6) (drill 0.3) (layers F.Cu B.Cu) (net 2))
+  (via (at 125 125) (size 0.6) (drill 0.3) (layers F.Cu B.Cu) (net 2))
+  (via (at 125 120) (size 0.6) (drill 0.3) (layers F.Cu B.Cu) (net 2))
+  (via (at 125 115) (size 0.6) (drill 0.3) (layers F.Cu B.Cu) (net 2))
+  (via (at 125 90) (size 0.6) (drill 0.3) (layers F.Cu B.Cu) (net 2))
+  (via (at 120 90) (size 0.6) (drill 0.3) (layers F.Cu B.Cu) (net 2))
+  (via (at 120 110) (size 0.6) (drill 0.3) (layers F.Cu B.Cu) (net 2))
+  (via (at 120 115) (size 0.6) (drill 0.3) (layers F.Cu B.Cu) (net 2))
+  (via (at 120 120) (size 0.6) (drill 0.3) (layers F.Cu B.Cu) (net 2))
+  (via (at 120 125) (size 0.6) (drill 0.3) (layers F.Cu B.Cu) (net 2))
+  (via (at 115 125) (size 0.6) (drill 0.3) (layers F.Cu B.Cu) (net 2))
+  (via (at 110 120) (size 0.6) (drill 0.3) (layers F.Cu B.Cu) (net 2))
+  (via (at 110 125) (size 0.6) (drill 0.3) (layers F.Cu B.Cu) (net 2))
+  (via (at 105 125) (size 0.6) (drill 0.3) (layers F.Cu B.Cu) (net 2))
+  (via (at 105 120) (size 0.6) (drill 0.3) (layers F.Cu B.Cu) (net 2))
+  (via (at 100 120) (size 0.6) (drill 0.3) (layers F.Cu B.Cu) (net 2))
+  (via (at 100 125) (size 0.6) (drill 0.3) (layers F.Cu B.Cu) (net 2))
+  (via (at 95 125) (size 0.6) (drill 0.3) (layers F.Cu B.Cu) (net 2))
+  (via (at 95 120) (size 0.6) (drill 0.3) (layers F.Cu B.Cu) (net 2))
+  (via (at 90 120) (size 0.6) (drill 0.3) (layers F.Cu B.Cu) (net 2))
+  (via (at 90 125) (size 0.6) (drill 0.3) (layers F.Cu B.Cu) (net 2))
+  (via (at 85 125) (size 0.6) (drill 0.3) (layers F.Cu B.Cu) (net 2))
   (via (at 92.35 104.55) (size 0.45) (drill 0.2) (layers F.Cu B.Cu) (net 24))
   (via (at 86 102.05) (size 0.45) (drill 0.2) (layers F.Cu B.Cu) (net 19))
