File: pcb/homebrew-computer/homebrew-computer.kicad_pcb (KiCad board)
At the start: 4 copper layers, 100 x 50 mm, 100 parts, among them J1 Conn_01x02_Male, J2 Conn_01x02_Male, J3 Conn_02x03_Counter_Clockwise, J4 Conn_02x20_Odd_Even, J5 Conn_01x04_Male, J6 Conn_01x02, SW1 SW_Push, U1 TLV73333PDBV, U10 74LVC16374ADGG,112, U11 74LVC16374ADGG,112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

Commit message: Add silkscreen
Parts:
- added REF**: ESD-Logo_6.6x6mm_SilkScreen, Symbol:ESD-Logo_6.6x6mm_SilkScreen, B.Cu at (52.0, 82.0)
- added REF**: WEEE-Logo_4.2x6mm_SilkScreen, Symbol:WEEE-Logo_4.2x6mm_SilkScreen, B.Cu at (45.0, 82.0)
Other:
- board text added: "EXT_CLK"
- board text added: "Ext_Clk"
- board text added: "Power"
- board text added: "Reset"
- board text added: "cchaine"

Commit message: Invert silkscreen on bottom
Parts:
- moved REF** 91.1 mm to (126.9, 122.0), turned to 180 degrees
- moved REF** 78.8 mm to (119.9, 122.0), turned to 180 degrees
Changed lines of the file:
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@@
   (general
     (thickness 1.6)
-    (drawings 27)
+    (drawings 21)
     (tracks 2008)
     (zones 0)
@@
     (add_net VCC)
   )
+  (module Button_Switch_SMD:Panasonic_EVQPUJ_EVQPUA (layer F.Cu)
+    (at 58 124 180)
+    (descr http://industrial.panasonic.com/cdbs/www-data/pdf/ATV0000/ATV0000CE5.pdf)
+    (tags "SMD SMT SPST EVQPUJ EVQPUA")
+    (attr smd)
+    (fp_text reference SW1 (at 0 -4.5 90) (layer F.Fab)
+      (effects (font (size 1 1) (thickness 0.15)))
+    )
+    (fp_text value SW_Push (at 0 3.5) (layer F.Fab)
+      (effects (font (size 1 1) (thickness 0.15)))
+    )
+    (fp_line (start 3.9 2.25) (end 3.9 -3.25) (layer F.CrtYd) (width 0.05))
+    (fp_line (start 2.35 -1.85) (end 1.425 -1.85) (layer F.SilkS) (width 0.12))
+    (fp_line (start 2.35 1.85) (end -2.35 1.85) (layer F.SilkS) (width 0.12))
+    (fp_line (start -2.45 0.275) (end -2.45 -0.275) (layer F.SilkS) (width 0.12))
+    (fp_line (start -1.3 -2.75) (end -1.3 -1.75) (layer F.Fab) (width 0.1))
+    (fp_line (start 1.3 -2.75) (end 1.3 -1.75) (layer F.Fab) (width 0.1))
+    (fp_line (start 1.3 -2.75) (end -1.3 -2.75) (layer F.Fab) (width 0.1))
+    (fp_line (start 2.35 1.75) (end 2.35 -1.75) (layer F.Fab) (width 0.1))
+    (fp_line (start -2.35 1.75) (end -2.35 -1.75) (layer F.Fab) (width 0.1))
+    (fp_line (start 2.35 -1.75) (end -2.35 -1.75) (layer F.Fab) (width 0.1))
+    (fp_line (start 2.35 1.75) (end -2.35 1.75) (layer F.Fab) (width 0.1))
+    (fp_line (start 2.45 0.275) (end 2.45 -0.275) (layer F.SilkS) (width 0.12))
+    (fp_line (start -1.425 -1.85) (end -2.35 -1.85) (layer F.SilkS) (width 0.12))
+    (fp_line (start -3.9 2.25) (end -3.9 -3.25) (layer F.CrtYd) (width 0.05))
+    (fp_line (start 3.9 2.25) (end -3.9 2.25) (layer F.CrtYd) (width 0.05))
+    (fp_line (start 3.9 -3.25) (end -3.9 -3.25) (layer F.CrtYd) (width 0.05))
+    (fp_text user %R (at 0 0) (layer F.Fab)
+      (effects (font (size 1 1) (thickness 0.15)))
+    )
+    (pad 1 smd rect (at 2.625 -0.85) (size 1.55 1) (layers F.Cu F.Paste F.Mask)
+      (net 3 +3V3))
+    (pad 1 smd rect (at -2.625 -0.85) (size 1.55 1) (layers F.Cu F.Paste F.Mask)
+      (net 3 +3V3))
+    (pad 2 smd rect (at -2.625 0.85) (size 1.55 1) (layers F.Cu F.Paste F.Mask)
+      (net 7 "Net-(D2-Pad2)"))
+    (pad 2 smd rect (at 2.625 0.85) (size 1.55 1) (layers F.Cu F.Paste F.Mask)
+      (net 7 "Net-(D2-Pad2)"))
+    (model ${KISYS3DMOD}/Button_Switch_SMD.3dshapes/Panasonic_EVQPUJ_EVQPUA.wrl
+      (at (xyz 0 0 0))
+      (scale (xyz 1 1 1))
+      (rotate (xyz 0 0 0))
+    )
+    (model ${KIPRJMOD}/libs/EVQPU-JA-02K.STEP
+      (at (xyz 0 0 0))
+      (scale (xyz 1 1 1))
+      (rotate (xyz -90 0 180))
+    )
+  )
   (module Symbol:ESD-Logo_6.6x6mm_SilkScreen (layer B.Cu)
-    (at 52 82)
+    (at 119.9 122 180)
     (descr "Electrostatic discharge Logo")
     (tags "Logo ESD")
@@
   )
   (module Symbol:WEEE-Logo_4.2x6mm_SilkScreen (layer B.Cu)
-    (at 45 82)
+    (at 126.9 122 180)
     (descr "Waste Electrical and Electronic Equipment Directive")
     (tags "Logo WEEE")
@@
     )
   )
-  (module Button_Switch_SMD:Panasonic_EVQPUJ_EVQPUA (layer F.Cu)
-    (at 58 124 180)
-    (descr http://industrial.panasonic.com/cdbs/www-data/pdf/ATV0000/ATV0000CE5.pdf)
-    (tags "SMD SMT SPST EVQPUJ EVQPUA")
-    (attr smd)
-    (fp_text reference SW1 (at 0 -4.5 90) (layer F.Fab)
-      (effects (font (size 1 1) (thickness 0.15)))
-    )
-    (fp_text value SW_Push (at 0 3.5) (layer F.Fab)
-      (effects (font (size 1 1) (thickness 0.15)))
-    )
-    (fp_line (start 3.9 2.25) (end 3.9 -3.25) (layer F.CrtYd) (width 0.05))
-    (fp_line (start 2.35 -1.85) (end 1.425 -1.85) (layer F.SilkS) (width 0.12))
-    (fp_line (start 2.35 1.85) (end -2.35 1.85) (layer F.SilkS) (width 0.12))
-    (fp_line (start -2.45 0.275) (end -2.45 -0.275) (layer F.SilkS) (width 0.12))
-    (fp_line (start -1.3 -2.75) (end -1.3 -1.75) (layer F.Fab) (width 0.1))
-    (fp_line (start 1.3 -2.75) (end 1.3 -1.75) (layer F.Fab) (width 0.1))
-    (fp_line (start 1.3 -2.75) (end -1.3 -2.75) (layer F.Fab) (width 0.1))
-    (fp_line (start 2.35 1.75) (end 2.35 -1.75) (layer F.Fab) (width 0.1))
-    (fp_line (start -2.35 1.75) (end -2.35 -1.75) (layer F.Fab) (width 0.1))
-    (fp_line (start 2.35 -1.75) (end -2.35 -1.75) (layer F.Fab) (width 0.1))
-    (fp_line (start 2.35 1.75) (end -2.35 1.75) (layer F.Fab) (width 0.1))
-    (fp_line (start 2.45 0.275) (end 2.45 -0.275) (layer F.SilkS) (width 0.12))
-    (fp_line (start -1.425 -1.85) (end -2.35 -1.85) (layer F.SilkS) (width 0.12))
-    (fp_line (start -3.9 2.25) (end -3.9 -3.25) (layer F.CrtYd) (width 0.05))
-    (fp_line (start 3.9 2.25) (end -3.9 2.25) (layer F.CrtYd) (width 0.05))
-    (fp_line (start 3.9 -3.25) (end -3.9 -3.25) (layer F.CrtYd) (width 0.05))
-    (fp_text user %R (at 0 0) (layer F.Fab)
-      (effects (font (size 1 1) (thickness 0.15)))
-    )
-    (pad 1 smd rect (at 2.625 -0.85) (size 1.55 1) (layers F.Cu F.Paste F.Mask)
-      (net 3 +3V3))
-    (pad 1 smd rect (at -2.625 -0.85) (size 1.55 1) (layers F.Cu F.Paste F.Mask)
-      (net 3 +3V3))
-    (pad 2 smd rect (at -2.625 0.85) (size 1.55 1) (layers F.Cu F.Paste F.Mask)
-      (net 7 "Net-(D2-Pad2)"))
-    (pad 2 smd rect (at 2.625 0.85) (size 1.55 1) (layers F.Cu F.Paste F.Mask)
-      (net 7 "Net-(D2-Pad2)"))
-    (model ${KISYS3DMOD}/Button_Switch_SMD.3dshapes/Panasonic_EVQPUJ_EVQPUA.wrl
-      (at (xyz 0 0 0))
-      (scale (xyz 1 1 1))
-      (rotate (xyz 0 0 0))
-    )
-    (model ${KIPRJMOD}/libs/EVQPU-JA-02K.STEP
-      (at (xyz 0 0 0))
-      (scale (xyz 1 1 1))
-      (rotate (xyz -90 0 180))
-    )
-  )
   (module Jumper:SolderJumper-2_P1.3mm_Open_RoundedPad1.0x1.5mm (layer B.Cu)
     (at 59.35 119 270)
@@
     )
   )
-  (gr_line (start 60.35 122.15) (end 60.35 122.55) (layer F.SilkS) (width 0.12))
-  (gr_line (start 55.65 122.15) (end 55.65 122.55) (layer F.SilkS) (width 0.12))
-  (gr_line (start 55.65 120.34) (end 55.65 122.15) (layer F.SilkS) (width 0.12))
-  (gr_line (start 60.35 120.34) (end 55.65 120.34) (layer F.SilkS) (width 0.12))
-  (gr_line (start 60.35 122.15) (end 60.35 120.34) (layer F.SilkS) (width 0.12))
-  (gr_text Reset (at 58 121.2 180) (layer F.SilkS)
-    (effects (font (size 0.75 0.75) (thickness 0.1875)))
-  )
   (gr_line (start 44.3 116.1) (end 41.985 116.11) (layer F.SilkS) (width 0.12))
   (gr_line (start 44.3 111.9) (end 44.3 116.1) (layer F.SilkS) (width 0.12))
@@
     (effects (font (size 0.75 0.75) (thickness 0.1875)))
   )
-  (gr_text EXT_CLK (at 54 118.8 180) (layer B.SilkS)
+  (gr_text EXT_CLK (at 54 119.2) (layer B.SilkS)
     (effects (font (size 1 1) (thickness 0.2)) (justify mirror))
   )
-  (gr_text cchaine (at 126.7 79.5 180) (layer B.SilkS)
+  (gr_text cchaine (at 45.3 124.5) (layer B.SilkS)
     (effects (font (size 1 1) (thickness 0.2)) (justify mirror))
   )

Commit message: Change connector for a more common one, and change the diode footprint
Parts:
- removed REF**: ESD-Logo_6.6x6mm_SilkScreen, Symbol:ESD-Logo_6.6x6mm_SilkScreen
- removed REF**: WEEE-Logo_4.2x6mm_SilkScreen, Symbol:WEEE-Logo_4.2x6mm_SilkScreen
- D2, D3, D4, D5, D6, D7, D8, D9: footprint Diode_SMD:D_0402_1005Metric_Pad0.77x0.64mm_HandSolder -> Diode_SMD:D_0603_1608Metric_Pad1.05x0.95mm_HandSolder
- J4: footprint Connector_Molex:Molex_Pico-Clasp_203566-4007_2x20_P1.00mm_Horizontal -> Connector_Molex:Micro-Lock-Plus-02x20
- moved D9 1.82 mm to (92.2, 89.0)
- moved D8 1.78 mm to (103.7, 89.0)
- moved D3 1.21 mm to (94.2, 89.0)
- moved D5 1.21 mm to (101.8, 89.0)
- moved J4 0.84 mm to (130.7, 102.0)
- moved D4 0.62 mm to (96.1, 89.0)
- moved D6 0.62 mm to (99.9, 89.0)
- moved D7 0.15 mm to (98.0, 89.0)
Routing:
- net /RESET: track 162.1 -> 156.9 mm
- net /IO_ADDR_IN: track 53.2 -> 56.4 mm
- net /IO/IO1: track 14.2 -> 11.7 mm
- net /IO/IO15: track 28.1 -> 30.6 mm
- net /IO/IO2: track 14.4 -> 12.0 mm
- net /IO/IO16: track 27.7 -> 30.0 mm
- net /IO/IO3: track 14.8 -> 12.6 mm
- net /IO/IO4: track 15.0 -> 12.9 mm
- net Net-(D3-Pad1): track 26.3 -> 28.4 mm
- net /IO_IN: track 52.4 -> 54.3 mm
- net /IO/IO5: track 15.5 -> 13.5 mm
- net /IO/IO6: track 15.7 -> 13.8 mm
- net /IO/IO7: track 16.1 -> 14.4 mm
- net /IO_OUT: track 53.8 -> 55.4 mm
- net /REG3_IN_L: track 11.6 -> 13.1 mm
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