File: pcb/computer-board/alu.sch (KiCad schematic (older format))
At the start: 4 parts, among them U4 XC9572XL-10VQG44C

Commit message: Rev A complete
Parts:
- U4: symbol homebrew-computer-rescue:XC9572XL-10VQG44C-XC9500XL -> computer-board-rescue:XC9572XL-10VQG44C-XC9500XL-homebrew-computer-rescue
Changed lines of the file:
@@
 OP_IN
 $Comp
-L homebrew-computer-rescue:XC9572XL-10VQG44C-XC9500XL U4
+L computer-board-rescue:XC9572XL-10VQG44C-XC9500XL-homebrew-computer-rescue U4
 U 1 1 5F975DA0
 P 2100 4100
@@
 $EndComp
 $Comp
-L homebrew-computer-rescue:XC9572XL-10VQG44C-XC9500XL U4
+L computer-board-rescue:XC9572XL-10VQG44C-XC9500XL-homebrew-computer-rescue U4
 U 2 1 5F97A638
 P 2100 1100
@@
 Connection ~ 2800 1400
 $Comp
-L homebrew-computer-rescue:XC9572XL-10VQG44C-XC9500XL U4
+L computer-board-rescue:XC9572XL-10VQG44C-XC9500XL-homebrew-computer-rescue U4
 U 3 1 5F97D3D1
 P 2850 1350
@@
 $EndComp
 $Comp
-L homebrew-computer-rescue:XC9572XL-10VQG44C-XC9500XL U4
+L computer-board-rescue:XC9572XL-10VQG44C-XC9500XL-homebrew-computer-rescue U4
 U 4 1 5F982A18
 P 5700 1050
@@
 $EndComp
 $Comp
-L homebrew-computer-rescue:XC9572XL-10VQG44C-XC9500XL U4
+L computer-board-rescue:XC9572XL-10VQG44C-XC9500XL-homebrew-computer-rescue U4
 U 5 1 5F987E07
 P 6200 1050
