File: pcb/computer-board/program_counter.sch (KiCad schematic (older format))
At the start: 4 parts, among them U8 XC9536XL-10VQG44C

Commit message: Rev A complete
Parts:
- U8: symbol homebrew-computer-rescue:XC9536XL-10VQG44C-XC9500XL -> computer-board-rescue:XC9536XL-10VQG44C-XC9500XL-homebrew-computer-rescue
Changed lines of the file:
@@
 Inputs/Outputs
 $Comp
-L homebrew-computer-rescue:XC9536XL-10VQG44C-XC9500XL U8
+L computer-board-rescue:XC9536XL-10VQG44C-XC9500XL-homebrew-computer-rescue U8
 U 1 1 5FA8CEAA
 P 3050 5750
@@
 $EndComp
 $Comp
-L homebrew-computer-rescue:XC9536XL-10VQG44C-XC9500XL U8
+L computer-board-rescue:XC9536XL-10VQG44C-XC9500XL-homebrew-computer-rescue U8
 U 2 1 5FA9060B
 P 2700 1050
@@
 Connection ~ 3400 1350
 $Comp
-L homebrew-computer-rescue:XC9536XL-10VQG44C-XC9500XL U8
+L computer-board-rescue:XC9536XL-10VQG44C-XC9500XL-homebrew-computer-rescue U8
 U 3 1 5FA92D8C
 P 3450 1300
@@
 $EndComp
 $Comp
-L homebrew-computer-rescue:XC9536XL-10VQG44C-XC9500XL U8
+L computer-board-rescue:XC9536XL-10VQG44C-XC9500XL-homebrew-computer-rescue U8
 U 5 1 5FA98EFF
 P 3300 2400
@@
 TDO
 $Comp
-L homebrew-computer-rescue:XC9536XL-10VQG44C-XC9500XL U8
+L computer-board-rescue:XC9536XL-10VQG44C-XC9500XL-homebrew-computer-rescue U8
 U 4 1 5FA96F85
 P 2800 2400
