File: modules/register-module/register-module.kicad_pcb (KiCad board)
At the start: 4 copper layers, 159.9 x 99.9 mm, 48 parts, among them J1 C96ABC, U1 74HC04, U10 74HC574, U11 74HC574, U12 74HC574, U13 74HC161, U14 74HC161, U15 74HC161, U16 74HC161, U17 74HC245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

Commit message: changed the mask clearance for plotting
Parts:
- R1: value R_Small -> 10k
Other:
- rule pad_to_mask_clearance: 0.2 -> 0
