File: pcb/power.kicad_sch (KiCad schematic)
At the start: 0 parts

Commit message: add power supply
Parts:
- added C? (x5): 100uF, symbol Device:C_Small
- added C? (x2): 22uF, symbol Device:C_Small
- added C? (x2): 47uF, symbol Device:C_Small
- added C? (x2): open, symbol Device:C_Small
- added C? (x2): 100nF, symbol Device:C_Small
- added C?: 2.2uF, symbol Device:C_Small
- added C?: 100uF, symbol Device:C_Polarized_Small
- added C? (x5): 0.1uF, symbol Device:C_Small
- added L?: 560nH, symbol Device:L_Iron
- added L?: 1.2uH, symbol Device:L_Iron
- added NT?: NetTie_2, symbol Device:NetTie_2
- added R?: 17.4k, symbol Device:R_Small
- added R? (x5): 10k, symbol Device:R_Small
- added R? (x2): 100k, symbol Device:R_Small
- added R?: 14k, symbol Device:R_Small
- added R?: 8k, symbol Device:R_Small
- added R?: 39.9k, symbol Device:R_Small
- added R?: 15.4k, symbol Device:R_Small
- added R?: 56k, symbol Device:R_Small
- added U?: TPS541620, symbol Regulator_Switching:TPS541620
Connections:
- new net: R?.1, R?.2, U?.10 (MODE2)
- new net: C?.1, R?.1, R?.2, U?.13 (FB1)
- new net: R?.1, U?.22 (PGOOD1)
- new net: C?.1, R?.1, R?.2, U?.17 (FB2/VSHARE)
- new net: R?.1, R?.1, U?.9 (MODE1)
- new net: R?.1, U?.21 (PGOOD2/CLKO)
- new net: C?.1, U?.1 (BOOT2)
- new net: C?.2, L?.1, U?.2 (SW2)
- new net: U?.24 (PVIN2), U?.6 (PVIN1)
- new net: C?.2, L?.1, U?.4 (SW1)
- new net: C?.1, U?.5 (BOOT1)
- new net +1V2: C?.1, C?.1, C?.1, C?.2, L?.2, R?.2
- new net +3V3: C?.1, C?.1, C?.2, L?.2, R?.1, R?.2
- new net BP5: C?.1, C?.1, R?.2, R?.2, U?.16 (BP5)
- new net EN1: R?.1, R?.2, U?.20 (EN1)
- new net EN2: R?.1, R?.2, U?.18 (EN2/ISHARE)
- new net GND: C?.2, C?.2, C?.2, C?.2, C?.2, C?.2, C?.2, C?.2, C?.2, C?.2, C?.2, C?.2, C?.2, C?.2, C?.2, C?.2, NT?.1, U?.14 (GOSNS), U?.23 (PGND), U?.25 (PGND), U?.3 (PGND), U?.7 (PGND)
- new net GND1: NT?.2, R?.1, R?.1, R?.2, R?.2, R?.2, R?.2, U?.15 (AGND)
- new net SS: U?.12 (SS)
- new net SYNC: U?.8 (SYNC)
- new net VCC: C?.1, C?.1, C?.1, C?.1, C?.1, C?.1, C?.1, C?.1, C?.1
Other:
- note added: "Inductor value Lo = ((Vin-Vout)/(K*Iout)) * (Vout / (Vin*fsw)) Iripple = ((Vinmax - Vout)/(Lo_eff) * (Vout / Vinmax*fsw)) RMS inductor current = sqrt( Iout^2 + (Iripple^2 / 12) ) Inductor peak current = Iout + Iripple / 2"
- note added: "Mode 1 -> 15.4k for 1.5pF ramp capacitor on VOUT2 Mode 2 -> 17.4k for 1MHz switching frequency and 1.5pF ramp capacitor on VOUT1"
- note added: "Mode selection :"
- note added: "Output inductor selection :"
- note added: "Output voltage Resistors Selection :"
- note added: "Rfb_t = Rfb_b * ((Vout - Vfb)/Vfb)"
- note added: "Sequencing and UVLO :"
- note added: "Vout2 first with UVLO from Vin -> Enable when Vin >= 6V Vout1 second from 3.3v -> Enable when 3.3v rail >= 2.7V"
