File: pcb/dram.kicad_sch (KiCad schematic)
At the start: 0 parts

Commit message: add the din connector
Parts:
- added C? (x14): 470nF, symbol Device:C_Small
- added C? (x2): 100uF, symbol Device:C_Small
- added C? (x2): 4.7uF, symbol Device:C_Small
- added U? (x2): IS42S16100H, symbol is42s16100h:IS42S16100H
Connections:
- new net +3V3: C?.1, C?.1, C?.1, C?.1, C?.1, C?.1, C?.1, C?.1, C?.1, C?.1, C?.1, C?.1, C?.1, C?.1, C?.1, C?.1, C?.1, C?.1, U?.A7 (VDD), U?.A7 (VDD), U?.B6 (VDDQ), U?.B6 (VDDQ), U?.C2 (VDDQ), U?.C2 (VDDQ), U?.E6 (VDDQ), U?.E6 (VDDQ), U?.F2 (VDDQ), U?.F2 (VDDQ), U?.H6 (VDD), U?.H6 (VDD), U?.R7 (VDD), U?.R7 (VDD)
- new net DRAM1_A0: U?.N6 (A0)
- new net DRAM1_A1: U?.P7 (A1)
- new net DRAM1_A10: U?.N7 (A10)
- new net DRAM1_A11: U?.M1 (A11)
- new net DRAM1_A2: U?.P6 (A2)
- new net DRAM1_A3: U?.R6 (A3)
- new net DRAM1_A4: U?.R2 (A4)
- new net DRAM1_A5: U?.P2 (A5)
- new net DRAM1_A6: U?.P1 (A6)
- new net DRAM1_A7: U?.N2 (A7)
- new net DRAM1_A8: U?.N1 (A8)
- new net DRAM1_A9: U?.M2 (A9)
- new net DRAM1_CAS#: U?.K7 (CAS#), U?.L1 (CKE)
- new net DRAM1_CS#: U?.L7 (CS#)
- new net DRAM1_IO0: U?.A6 (DQ0)
- new net DRAM1_IO1: U?.B7 (DQ1)
- new net DRAM1_IO10: U?.E1 (DQ10)
- new net DRAM1_IO11: U?.D2 (DQ11)
- new net DRAM1_IO12: U?.D1 (DQ12)
- new net DRAM1_IO13: U?.C1 (DQ13)
- new net DRAM1_IO14: U?.B1 (DQ14)
- new net DRAM1_IO15: U?.A2 (DQ15)
- new net DRAM1_IO2: U?.C7 (DQ2)
- new net DRAM1_IO3: U?.D7 (DQ3)
- new net DRAM1_IO4: U?.D6 (DQ4)
- new net DRAM1_IO5: U?.E7 (DQ5)
- new net DRAM1_IO6: U?.F7 (DQ6)
- new net DRAM1_IO7: U?.G7 (DQ7)
- new net DRAM1_IO8: U?.G1 (DQ8)
- new net DRAM1_IO9: U?.F1 (DQ9)
- new net DRAM1_LDQM: U?.J6 (LDQM)
- new net DRAM1_RAS#: U?.K6 (RAS#)
- new net DRAM1_UDQM: U?.J2 (UDQM)
- new net DRAM1_WE#: U?.J7 (WE#)
- new net DRAM2_A0: U?.N6 (A0)
- new net DRAM2_A1: U?.P7 (A1)
- new net DRAM2_A10: U?.N7 (A10)
- new net DRAM2_A11: U?.M1 (A11)
- new net DRAM2_A2: U?.P6 (A2)
- new net DRAM2_A3: U?.R6 (A3)
- new net DRAM2_A4: U?.R2 (A4)
- new net DRAM2_A5: U?.P2 (A5)
- new net DRAM2_A6: U?.P1 (A6)
- new net DRAM2_A7: U?.N2 (A7)
- new net DRAM2_A8: U?.N1 (A8)
- new net DRAM2_A9: U?.M2 (A9)
- new net DRAM2_CAS#: U?.K7 (CAS#), U?.L1 (CKE)
- new net DRAM2_CS#: U?.L7 (CS#)
- new net DRAM2_IO0: U?.A6 (DQ0)
- new net DRAM2_IO1: U?.B7 (DQ1)
- new net DRAM2_IO10: U?.E1 (DQ10)
- new net DRAM2_IO11: U?.D2 (DQ11)
- new net DRAM2_IO12: U?.D1 (DQ12)
- new net DRAM2_IO13: U?.C1 (DQ13)
- new net DRAM2_IO14: U?.B1 (DQ14)
- new net DRAM2_IO15: U?.A2 (DQ15)
- new net DRAM2_IO2: U?.C7 (DQ2)
- new net DRAM2_IO3: U?.D7 (DQ3)
- new net DRAM2_IO4: U?.D6 (DQ4)
- new net DRAM2_IO5: U?.E7 (DQ5)
- new net DRAM2_IO6: U?.F7 (DQ6)
- new net DRAM2_IO7: U?.G7 (DQ7)
- new net DRAM2_IO8: U?.G1 (DQ8)
- new net DRAM2_IO9: U?.F1 (DQ9)
- new net DRAM2_LDQM: U?.J6 (LDQM)
- new net DRAM2_RAS#: U?.K6 (RAS#)
- new net DRAM2_UDQM: U?.J2 (UDQM)
- new net DRAM2_WE#: U?.J7 (WE#)
- new net DRAM_CLK: U?.K2 (CLK), U?.K2 (CLK)
- new net GND: C?.2, C?.2, C?.2, C?.2, C?.2, C?.2, C?.2, C?.2, C?.2, C?.2, C?.2, C?.2, C?.2, C?.2, C?.2, C?.2, C?.2, C?.2, U?.A1 (GND), U?.A1 (GND), U?.B2 (GND), U?.B2 (GND), U?.C6 (GNDQ), U?.C6 (GNDQ), U?.E2 (GNDQ), U?.E2 (GNDQ), U?.F6 (GNDQ), U?.F6 (GNDQ), U?.R1 (GND), U?.R1 (GND)

Commit message: start associating footprints
Parts:
- C72: renamed from C?; footprint (none) -> Capacitor_SMD:CP_Elec_6.3x7.7; Ref (none) -> GYA1E101MCW1GS
- C73: renamed from C?; footprint (none) -> Capacitor_SMD:CP_Elec_4x4.5; Ref (none) -> EDK475M025A9BAA
- C74, C75, C76, C77, C78, C79, C80, C83, C84, C85, C86, C87, C88, C89: renamed from C?; footprint (none) -> Capacitor_SMD:C_0402_1005Metric
- C81: renamed from C?; footprint (none) -> Capacitor_SMD:C_Elec_6.3x7.7
- C82: renamed from C?; footprint (none) -> Capacitor_SMD:CP_Elec_4x4.5
- gave numbers to parts that had none: 2

Commit message: add tps541620 footprint
Parts:
- U12: footprint (none) -> Package_BGA:IS42S16100H; Ref (none) -> IS42S16100H-7BL
- U13: footprint (none) -> Package_BGA:IS42S16100H
Changed lines of the file:
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@@
     (property "Reference" "U12" (id 0) (at 182.88 30.48 0))
     (property "Value" "IS42S16100H" (id 1) (at 182.88 33.02 0))
-    (property "Footprint" "" (id 2) (at 167.64 34.29 0)
+    (property "Footprint" "Package_BGA:IS42S16100H" (id 2) (at 167.64 34.29 0)
       (effects (font (size 1.27 1.27)) hide)
     )
     (property "Datasheet" "" (id 3) (at 167.64 34.29 0)
       (effects (font (size 1.27 1.27)) hide)
+    )
+    (property "Ref" "IS42S16100H-7BL " (id 4) (at 182.88 27.94 0)
+      (effects (font (size 0.5 0.5)))
     )
     (pin "A1")
@@
     (property "Reference" "U13" (id 0) (at 257.81 30.48 0))
     (property "Value" "IS42S16100H" (id 1) (at 257.81 33.02 0))
-    (property "Footprint" "" (id 2) (at 242.57 34.29 0)
+    (property "Footprint" "Package_BGA:IS42S16100H" (id 2) (at 242.57 34.29 0)
       (effects (font (size 1.27 1.27)) hide)
     )

Commit message: add components to pcb
Parts:
- U12, U13: footprint Package_BGA:IS42S16100H -> IS42S16100H:IS42S16100H
Changed lines of the file:
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@@
-(kicad_sch (version 20210126) (generator eeschema)
+(kicad_sch (version 20210406) (generator eeschema)
   (paper "User" 299.999 159.995)
   (junction (at 33.02 44.45) (diameter 0.9144) (color 0 0 0 0))
@@
     (property "Reference" "U12" (id 0) (at 182.88 30.48 0))
     (property "Value" "IS42S16100H" (id 1) (at 182.88 33.02 0))
-    (property "Footprint" "Package_BGA:IS42S16100H" (id 2) (at 167.64 34.29 0)
+    (property "Footprint" "IS42S16100H:IS42S16100H" (id 2) (at 167.64 34.29 0)
       (effects (font (size 1.27 1.27)) hide)
     )
@@
     (property "Reference" "U13" (id 0) (at 257.81 30.48 0))
     (property "Value" "IS42S16100H" (id 1) (at 257.81 33.02 0))
-    (property "Footprint" "Package_BGA:IS42S16100H" (id 2) (at 242.57 34.29 0)
-      (effects (font (size 1.27 1.27)) hide)
-    )
+    (property "Footprint" "IS42S16100H:IS42S16100H" (id 2) (at 242.57 34.29 0)
+      (effects (font (size 1.27 1.27)) hide)
+    )
