File: pcb/board.kicad_sch (KiCad schematic)
At the start: 4 parts

Commit message: add 3d files to some footprints
Parts:
- removed MK2, MK4: Mounting_Hole_PAD, Mounting_Holes:MountingHole_2.7mm, symbol EuroCard160mmX100mm_holes:Mounting_Hole_PAD-Mechanical
Connections:
- no-connect marks 4 -> 2
Changed lines of the file:
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@@
   (paper "User" 180.01 140.005)
   (no_connect (at 26.67 97.79))
-  (no_connect (at 26.67 105.41))
   (no_connect (at 26.67 113.03))
-  (no_connect (at 26.67 120.65))
   (symbol (lib_id "EuroCard160mmX100mm_holes:Mounting_Hole_PAD-Mechanical") (at 26.67 95.25 0) (unit 1)
     (in_bom yes) (on_board yes)
@@
     (pin "1")
   )
-  (symbol (lib_id "EuroCard160mmX100mm_holes:Mounting_Hole_PAD-Mechanical") (at 26.67 102.87 0) (unit 1)
-    (in_bom yes) (on_board yes)
-    (property "Reference" "MK2" (id 0) (at 29.21 101.5746 0)
-      (effects (font (size 1.27 1.27)) (justify left))
-    )
-    (property "Value" "Mounting_Hole_PAD" (id 1) (at 29.21 103.886 0)
-      (effects (font (size 1.27 1.27)) (justify left))
-    )
-    (property "Footprint" "Mounting_Holes:MountingHole_2.7mm" (id 2) (at 26.67 102.87 0)
-      (effects (font (size 1.27 1.27)) hide)
-    )
-    (property "Datasheet" "" (id 3) (at 26.67 102.87 0)
-      (effects (font (size 1.27 1.27)) hide)
-    )
-    (pin "1")
-  )
   (symbol (lib_id "EuroCard160mmX100mm_holes:Mounting_Hole_PAD-Mechanical") (at 26.67 110.49 0) (unit 1)
     (in_bom yes) (on_board yes)
@@
     )
     (property "Datasheet" "" (id 3) (at 26.67 110.49 0)
-      (effects (font (size 1.27 1.27)) hide)
-    )
-    (pin "1")
-  )
-  (symbol (lib_id "EuroCard160mmX100mm_holes:Mounting_Hole_PAD-Mechanical") (at 26.67 118.11 0) (unit 1)
-    (in_bom yes) (on_board yes)
-    (property "Reference" "MK4" (id 0) (at 29.21 116.8146 0)
-      (effects (font (size 1.27 1.27)) (justify left))
-    )
-    (property "Value" "Mounting_Hole_PAD" (id 1) (at 29.21 119.126 0)
-      (effects (font (size 1.27 1.27)) (justify left))
-    )
-    (property "Footprint" "Mounting_Holes:MountingHole_2.7mm" (id 2) (at 26.67 118.11 0)
-      (effects (font (size 1.27 1.27)) hide)
-    )
-    (property "Datasheet" "" (id 3) (at 26.67 118.11 0)
       (effects (font (size 1.27 1.27)) hide)
     )
@@
       (reference "MK1") (unit 1) (value "Mounting_Hole_PAD") (footprint "Mounting_Holes:MountingHole_2.7mm")
     )
-    (path "/00000000-0000-0000-0000-00005a6cff98"
-      (reference "MK2") (unit 1) (value "Mounting_Hole_PAD") (footprint "Mounting_Holes:MountingHole_2.7mm")
-    )
     (path "/00000000-0000-0000-0000-00005a6cfffa"
       (reference "MK3") (unit 1) (value "Mounting_Hole_PAD") (footprint "Mounting_Holes:MountingHole_2.7mm")
     )
-    (path "/00000000-0000-0000-0000-00005a6d003f"
-      (reference "MK4") (unit 1) (value "Mounting_Hole_PAD") (footprint "Mounting_Holes:MountingHole_2.7mm")
-    )
     (path "/deae845a-ed89-4dc8-b611-a45627046b99/02794d2e-5473-4454-accb-f831861c1aa3"
