File: pcb/usb.kicad_sch (KiCad schematic)
At the start: 47 parts, among them J1 Conn_02x03_Counter_Clockwise, J2 USB_B, U6 74LVC1G04, U7 SN74AVC4T245PW, U8 FT2232HQ, U9 93LCxxBxxOT, Y1 12MHz

Commit message: place components relative to each others
Parts:
- removed C47: 0.1u, Capacitor_SMD:C_0402_1005Metric, symbol Device:C_Small
Connections:
- net +3V3: now also C34.1, U8.12 (VCORE), U8.37 (VCORE), U8.49 (VREGOUT), U8.64 (VCORE)
Changed lines of the file:
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@@
   (junction (at 41.91 143.51) (diameter 1.016) (color 0 0 0 0))
   (junction (at 43.18 54.61) (diameter 0.9144) (color 0 0 0 0))
+  (junction (at 50.8 34.29) (diameter 0.9144) (color 0 0 0 0))
   (junction (at 50.8 39.37) (diameter 1.016) (color 0 0 0 0))
   (junction (at 50.8 76.2) (diameter 1.016) (color 0 0 0 0))
@@
   (junction (at 52.07 116.84) (diameter 0.9144) (color 0 0 0 0))
   (junction (at 52.07 121.92) (diameter 0.9144) (color 0 0 0 0))
-  (junction (at 52.07 138.43) (diameter 0.9144) (color 0 0 0 0))
   (junction (at 59.69 76.2) (diameter 1.016) (color 0 0 0 0))
   (junction (at 59.69 97.79) (diameter 1.016) (color 0 0 0 0))
@@
     (stroke (width 0) (type solid) (color 0 0 0 0))
   )
-  (wire (pts (xy 41.91 138.43) (xy 52.07 138.43))
+  (wire (pts (xy 41.91 138.43) (xy 62.23 138.43))
     (stroke (width 0) (type solid) (color 0 0 0 0))
   )
@@
     (stroke (width 0) (type solid) (color 0 0 0 0))
   )
-  (wire (pts (xy 41.91 143.51) (xy 52.07 143.51))
-    (stroke (width 0) (type solid) (color 0 0 0 0))
-  )
   (wire (pts (xy 43.18 54.61) (xy 52.07 54.61))
     (stroke (width 0) (type solid) (color 0 0 0 0))
@@
     (stroke (width 0) (type solid) (color 0 0 0 0))
   )
+  (wire (pts (xy 50.8 34.29) (xy 59.69 34.29))
+    (stroke (width 0) (type solid) (color 0 0 0 0))
+  )
   (wire (pts (xy 50.8 39.37) (xy 50.8 40.64))
     (stroke (width 0) (type solid) (color 0 0 0 0))
@@
     (stroke (width 0) (type solid) (color 0 0 0 0))
   )
-  (wire (pts (xy 52.07 138.43) (xy 62.23 138.43))
-    (stroke (width 0) (type solid) (color 0 0 0 0))
-  )
   (wire (pts (xy 59.69 76.2) (xy 67.31 76.2))
     (stroke (width 0) (type solid) (color 0 0 0 0))
@@
   )
   (wire (pts (xy 207.01 168.91) (xy 209.55 168.91))
+    (stroke (width 0) (type solid) (color 0 0 0 0))
+  )
+  (wire (pts (xy 209.55 38.1) (xy 209.55 52.07))
     (stroke (width 0) (type solid) (color 0 0 0 0))
   )
@@
     (effects (font (size 1.27 1.27)) (justify right bottom))
   )
+  (label "VCORE" (at 59.69 34.29 0)
+    (effects (font (size 1.27 1.27)) (justify left bottom))
+  )
   (label "JTAG_BUF_VCC" (at 62.23 138.43 0)
     (effects (font (size 1.27 1.27)) (justify left bottom))
@@
   )
   (label "VPHY" (at 196.85 43.18 180)
+    (effects (font (size 1.27 1.27)) (justify right bottom))
+  )
+  (label "VCORE" (at 209.55 38.1 180)
     (effects (font (size 1.27 1.27)) (justify right bottom))
   )
@@
       (effects (font (size 1.27 1.27)) hide)
     )
-    (pin "1")
-    (pin "2")
-  )
-  (symbol (lib_id "Device:C_Small") (at 52.07 140.97 0) (unit 1)
-    (in_bom yes) (on_board yes)
-    (property "Reference" "C47" (id 0) (at 54.61 140.3349 0)
-      (effects (font (size 1.27 1.27)) (justify left))
-    )
-    (property "Value" "0.1u" (id 1) (at 54.61 142.8749 0)
-      (effects (font (size 1.27 1.27)) (justify left))
-    )
-    (property "Footprint" "Capacitor_SMD:C_0402_1005Metric" (id 2) (at 52.07 140.97 0)
-      (effects (font (size 1.27 1.27)) hide)
-    )
-    (property "Datasheet" "~" (id 3) (at 52.07 140.97 0)
-      (effects (font (size 1.27 1.27)) hide)
-    )

Commit message: added silkscreen values
Parts:
- J1: footprint Connector_PinHeader_2.00mm:PinHeader_1x06_P2.00mm_Vertical -> Connector_IDC:IDC-Header_2x03_P2.54mm_Horizontal
Changed lines of the file:
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@@
       (effects (font (size 1.27 1.27)) hide)
     )
-    (property "Footprint" "Connector_PinHeader_2.00mm:PinHeader_1x06_P2.00mm_Vertical" (id 2) (at 351.79 43.18 0)
+    (property "Footprint" "Connector_IDC:IDC-Header_2x03_P2.54mm_Horizontal" (id 2) (at 351.79 43.18 0)
       (effects (font (size 1.27 1.27)) hide)
     )
